File: sheets/rom.kicad_sch (KiCad schematic)
At the start: 3 parts, among them U34 NEO-E0, U35 74LS259, U36 27C1024

Commit message: Merged in schematics from stable with footprints
Parts:
- U34: footprint (none) -> Package_LCC:PLCC-84
- U35: footprint (none) -> Package_DIP:DIP-16_W7.62mm
