File: sheets/z80_audio.kicad_sch (KiCad schematic)
At the start: 4 parts, among them U22 NEO-D0, U23 HM6116ASP-20, U24 Z80CPU

Commit message: Resistor Value Ω added
Parts:
- R30: value 4.7K -> 4.7KΩ
Changed lines of the file:
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@@
       (effects (font (size 1.27 1.27)) (justify left))
     )
-    (property "Value" "4.7K" (id 1) (at 140.208 51.0539 0)
+    (property "Value" "4.7KΩ" (id 1) (at 140.208 51.0539 0)
       (effects (font (size 1.27 1.27)) (justify left))
     )

Commit message: Assigning Footprints
Assigned some footprints to some components. Can still be wrong size on caps
Parts:
- R30: footprint (none) -> 1_NeoGeoLibrary:Resistor1-5mm
Changed lines of the file:
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@@
       (effects (font (size 1.27 1.27)) (justify left))
     )
-    (property "Footprint" "" (id 2) (at 138.684 49.784 0)
+    (property "Footprint" "1_NeoGeoLibrary:Resistor1-5mm" (id 2) (at 138.684 49.784 0)
       (effects (font (size 1.27 1.27)) hide)
     )

Commit message: Updated Footprints
Parts:
- U22: footprint (none) -> Package_LCC:PLCC-84
- U24: footprint (none) -> Package_DIP:DIP-40_W7.62mm
Changed lines of the file:
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@@
     (property "Reference" "U24" (id 0) (at 147.066 55.626 0))
     (property "Value" "Z80CPU" (id 1) (at 159.004 126.746 0))
-    (property "Footprint" "" (id 2) (at 159.004 81.026 0)
+    (property "Footprint" "Package_DIP:DIP-40_W7.62mm" (id 2) (at 159.004 81.026 0)
       (effects (font (size 1.27 1.27)) hide)
     )
@@
     (property "Reference" "U22" (id 0) (at 254.508 142.24 0))
     (property "Value" "NEO-D0" (id 1) (at 262.636 235.712 0))
-    (property "Footprint" "" (id 2) (at 262.636 201.676 0)
+    (property "Footprint" "Package_LCC:PLCC-84" (id 2) (at 262.636 201.676 0)
       (effects (font (size 1.27 1.27)) hide)
     )
