File: sheets/z80_audio.kicad_sch (KiCad schematic)
At the start: 4 parts, among them U22 NEO-D0, U23 HM6116ASP-20, U24 Z80CPU

Commit message: Merged in schematics from stable with footprints
Parts:
- U22: footprint (none) -> Package_LCC:PLCC-84
- U24: footprint (none) -> Package_DIP:DIP-40_W7.62mm

Commit message: Changed Z80 FootPrint
Parts:
- U24: footprint Package_DIP:DIP-40_W7.62mm -> Package_DIP:DIP-40_W15.24mm
Changed lines of the file:
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@@
     (property "Reference" "U24" (id 0) (at 147.066 55.626 0))
     (property "Value" "Z80CPU" (id 1) (at 159.004 126.746 0))
-    (property "Footprint" "Package_DIP:DIP-40_W7.62mm" (id 2) (at 159.004 81.026 0)
+    (property "Footprint" "Package_DIP:DIP-40_W15.24mm" (id 2) (at 159.004 81.026 0)
       (effects (font (size 1.27 1.27)) hide)
     )

Commit message: Sync footprints from Nightly Build
Parts:
- U22: footprint Package_LCC:PLCC-84 -> 1_NeoGeoLibrary:NEO-G0
- U23: footprint Package_DIP:DIP-28_W15.24mm -> Package_DIP:DIP-24_W7.62mm
Changed lines of the file:
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@@
     (property "Reference" "U22" (id 0) (at 254.508 142.24 0))
     (property "Value" "NEO-D0" (id 1) (at 262.636 235.712 0))
-    (property "Footprint" "Package_LCC:PLCC-84" (id 2) (at 262.636 201.676 0)
+    (property "Footprint" "1_NeoGeoLibrary:NEO-G0" (id 2) (at 262.636 201.676 0)
       (effects (font (size 1.27 1.27)) hide)
     )
@@
       (effects (font (size 1.27 1.27)) (justify left))
     )
-    (property "Footprint" "Package_DIP:DIP-28_W15.24mm" (id 2) (at 258.572 114.046 0)
+    (property "Footprint" "Package_DIP:DIP-24_W7.62mm" (id 2) (at 258.572 114.046 0)
       (effects (font (size 1.27 1.27)) hide)
     )

Commit message: Schematics Footprint updates
Parts:
- U23: footprint Package_DIP:DIP-24_W7.62mm -> 1_NeoGeoLibrary:DIP-24_W7.62mm
- U24: footprint Package_DIP:DIP-40_W15.24mm -> 1_NeoGeoLibrary:DIP-40_W15.24mm
Changed lines of the file:
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@@
       (effects (font (size 1.27 1.27)))
     )
-    (property "Footprint" "Package_DIP:DIP-40_W15.24mm" (at 159.004 81.026 0)
+    (property "Footprint" "1_NeoGeoLibrary:DIP-40_W15.24mm" (at 159.004 81.026 0)
       (effects (font (size 1.27 1.27)) hide)
     )
@@
       (effects (font (size 1.27 1.27)) (justify left))
     )
-    (property "Footprint" "Package_DIP:DIP-24_W7.62mm" (at 258.572 114.046 0)
+    (property "Footprint" "1_NeoGeoLibrary:DIP-24_W7.62mm" (at 258.572 114.046 0)
       (effects (font (size 1.27 1.27)) hide)
     )

Commit message: Some tweaks
Other:
- company: (none) -> SNK
- title: (none) -> NeoGeo AES
Changed lines of the file:
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@@
 (kicad_sch (version 20230121) (generator eeschema)
   (paper "A3")
+  (title_block
+    (title "NeoGeo AES")
+    (date "2023-08-19")
+    (rev "3.5")
+    (company "SNK")
+    (comment 3 "https://github.com/Board-Folk")
+    (comment 4 "Recreated By The Board Folk Team")
+  )
   (junction (at 281.432 229.616) (diameter 0) (color 0 0 0 0)
   )

Commit message: Updates to PCB Move P2 Joystick Port Move Memory Card Move Holes at top right Silkscreen added Update Titles
Other:
- title: NeoGeo AES -> NeoGeo AES 3-5
Changed lines of the file:
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@@
   (paper "A3")
   (title_block
-    (title "NeoGeo AES")
-    (date "2023-08-19")
-    (rev "3.5")
+    (title "NeoGeo AES 3-5")
+    (date "2023-08-27")
+    (rev "BF1.1")
     (company "SNK")
     (comment 3 "https://github.com/Board-Folk")
