File: sheets/clock.kicad_sch (KiCad schematic)
At the start: 28 parts, among them U39 CX23065A, U8 74HC04, U80 74HC04, X1 24.167829MHz, X2 3.579545MHz

Commit message: Sync Footprints from Nightly
Parts:
- C48, C51, C53, C54, C64: footprint 1_NeoGeoLibrary:CAP1-5mm -> 1_NeoGeoLibrary:CAP3-5mm
- C49: footprint 1_NeoGeoLibrary:CAP1-5mm -> 1_NeoGeoLibrary:CAP2-2.5mm
- TP1: footprint TestPoint:TestPoint_Pad_D4.0mm -> TestPoint:TestPoint_Pad_D1.5mm
- TP2: footprint TestPoint:TestPoint_Pad_D4.0mm -> TestPoint:TestPoint_THTPad_D1.5mm_Drill0.7mm
Changed lines of the file:
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@@
       (effects (font (size 1.27 1.27)) (justify right))
     )
-    (property "Footprint" "1_NeoGeoLibrary:CAP1-5mm" (id 2) (at 132.715 135.255 0)
+    (property "Footprint" "1_NeoGeoLibrary:CAP3-5mm" (id 2) (at 132.715 135.255 0)
       (effects (font (size 1.27 1.27)) hide)
     )
@@
       (effects (font (size 1.27 1.27)) (justify right))
     )
-    (property "Footprint" "1_NeoGeoLibrary:CAP1-5mm" (id 2) (at 92.71 175.895 0)
+    (property "Footprint" "1_NeoGeoLibrary:CAP3-5mm" (id 2) (at 92.71 175.895 0)
       (effects (font (size 1.27 1.27)) hide)
     )
@@
       (effects (font (size 1.27 1.27)) (justify right))
     )
-    (property "Footprint" "TestPoint:TestPoint_Pad_D4.0mm" (id 2) (at 172.72 173.355 0)
+    (property "Footprint" "TestPoint:TestPoint_THTPad_D1.5mm_Drill0.7mm" (id 2) (at 172.72 173.355 0)
       (effects (font (size 1.27 1.27)) hide)
     )
@@
       (effects (font (size 1.27 1.27)) (justify right))
     )
-    (property "Footprint" "1_NeoGeoLibrary:CAP1-5mm" (id 2) (at 173.99 135.255 0)
+    (property "Footprint" "1_NeoGeoLibrary:CAP3-5mm" (id 2) (at 173.99 135.255 0)
       (effects (font (size 1.27 1.27)) hide)
     )
@@
       (effects (font (size 1.27 1.27)) (justify right))
     )
-    (property "Footprint" "1_NeoGeoLibrary:CAP1-5mm" (id 2) (at 236.22 165.735 0)
+    (property "Footprint" "1_NeoGeoLibrary:CAP3-5mm" (id 2) (at 236.22 165.735 0)
       (effects (font (size 1.27 1.27)) hide)
     )
@@
     (property "Reference" "C53" (id 0) (at 158.115 90.17 90))
     (property "Value" "30pF" (id 1) (at 158.115 95.885 90))
-    (property "Footprint" "1_NeoGeoLibrary:CAP1-5mm" (id 2) (at 158.115 92.71 0)
+    (property "Footprint" "1_NeoGeoLibrary:CAP3-5mm" (id 2) (at 158.115 92.71 0)
       (effects (font (size 1.27 1.27)) hide)
     )
@@
       (effects (font (size 1.27 1.27)) (justify left))
     )
-    (property "Footprint" "1_NeoGeoLibrary:CAP1-5mm" (id 2) (at 222.885 175.895 0)
+    (property "Footprint" "1_NeoGeoLibrary:CAP2-2.5mm" (id 2) (at 222.885 175.895 0)
       (effects (font (size 1.27 1.27)) hide)
     )
@@
       (effects (font (size 1.27 1.27)) (justify left))
     )
-    (property "Footprint" "TestPoint:TestPoint_Pad_D4.0mm" (id 2) (at 324.866 108.966 0)
-      (effects (font (size 1.27 1.27)) hide)
-    )
+    (property "Footprint" "TestPoint:TestPoint_Pad_D1.5mm" (id 2) (at 324.866 108.966 0)
+      (effects (font (size 1.27 1.27)) hide)
+    )
