File: sheets/clock.kicad_sch (KiCad schematic)
At the start: 28 parts, among them U39 CX23065A, U8 74HC04, U80 74HC04, X1 24.167829MHz, X2 3.579545MHz

Commit message: More silkscreen tidy up, adding mouser components to BOM
Parts:
- R68: value 10KΩ -> 10K
- R70, R72: value 1MΩ -> 1M
- R71: value 10Ω -> 10
- R74: value 220KΩ -> 220K
Changed lines of the file:
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@@
       (effects (font (size 1.27 1.27)))
     )
-    (property "Value" "10KΩ" (at 191.135 175.26 90)
+    (property "Value" "10K" (at 191.135 175.26 90)
       (effects (font (size 1.27 1.27)))
     )
@@
       (effects (font (size 1.27 1.27)))
     )
-    (property "Value" "1MΩ" (at 260.096 102.616 90)
+    (property "Value" "1M" (at 260.096 102.616 90)
       (effects (font (size 1.27 1.27)))
     )
@@
       (effects (font (size 1.27 1.27)) (justify left))
     )
-    (property "Value" "10Ω" (at 224.155 156.845 0)
+    (property "Value" "10" (at 224.155 156.845 0)
       (effects (font (size 1.27 1.27)) (justify left))
     )
@@
       (effects (font (size 1.27 1.27)))
     )
-    (property "Value" "1MΩ" (at 143.51 115.57 90)
+    (property "Value" "1M" (at 143.51 115.57 90)
       (effects (font (size 1.27 1.27)))
     )
@@
       (effects (font (size 1.27 1.27)) (justify left))
     )
-    (property "Value" "220KΩ" (at 224.155 165.1 0)
+    (property "Value" "220K" (at 224.155 165.1 0)
       (effects (font (size 1.27 1.27)) (justify left))
     )

Commit message: Little tweaks to silkscreen Updated BOM with mouser parts
Parts:
- D3, D4, TC1, U39, X1: Comment (none) -> Use Original
- R101, R102: Mouser (none) -> 71-RN60E1003F
- R68: Mouser (none) -> 71-RN60E1002F
- R70, R72: Mouser (none) -> 71-RN60D-F-1M/R
- R71: Mouser (none) -> 71-CMF5010R000FHEK
- R74: Mouser (none) -> 71-RN60D2203F
- TP1, TP2: now left out of the parts list
- U8, U80: Mouser (none) -> 595-SN74HC04N
- X2: Mouser (none) -> 815-AB-3.579545-B2
Changed lines of the file:
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@@
     (title "NeoGeo AES 3-5")
     (date "2023-08-27")
-    (rev "BF1.1")
+    (rev "BF1.2")
     (company "SNK")
     (comment 3 "https://github.com/Board-Folk")
@@
       (effects (font (size 1.27 1.27)) hide)
     )
-    (property "Mouser" "" (at 191.135 173.355 0)
+    (property "Mouser" "71-RN60E1002F" (at 191.135 173.355 0)
+      (effects (font (size 1.27 1.27)) hide)
+    )
+    (property "Alternative" "" (at 191.135 173.355 0)
       (effects (font (size 1.27 1.27)) hide)
     )
@@
       (effects (font (size 1.27 1.27)) hide)
     )
-    (property "Mouser" "" (at 260.096 100.711 0)
+    (property "Mouser" "71-RN60D-F-1M/R" (at 260.096 100.711 0)
+      (effects (font (size 1.27 1.27)) hide)
+    )
+    (property "Alternative" "" (at 260.096 100.711 0)
       (effects (font (size 1.27 1.27)) hide)
     )
@@
       (effects (font (size 1.27 1.27)) hide)
     )
-    (property "Mouser" "" (at 312.166 115.316 0)
+    (property "Mouser" "595-SN74HC04N" (at 312.166 115.316 0)
+      (effects (font (size 1.27 1.27)) hide)
+    )
+    (property "Alternative" "" (at 312.166 115.316 0)
       (effects (font (size 1.27 1.27)) hide)
     )
@@
       (effects (font (size 1.27 1.27)) hide)
     )
+    (property "Alternative" "" (at 132.715 135.255 0)
+      (effects (font (size 1.27 1.27)) hide)
+    )
     (pin "1")
     (pin "2")
@@
       (effects (font (size 1.27 1.27)) hide)
     )
-    (property "Mouser" "" (at 111.76 108.585 0)
+    (property "Mouser" "71-RN60E1003F" (at 111.76 108.585 0)
+      (effects (font (size 1.27 1.27)) hide)
+    )
+    (property "Alternative" "" (at 111.76 108.585 0)
       (effects (font (size 1.27 1.27)) hide)
     )
@@
       (effects (font (size 1.27 1.27)) hide)
     )
+    (property "Comment" "Use Original" (at 132.715 102.87 0)
+      (effects (font (size 1.27 1.27)) hide)
+    )
+    (property "Alternative" "" (at 132.715 102.87 0)
+      (effects (font (size 1.27 1.27)) hide)
+    )
     (pin "0")
     (pin "1")
@@
       (effects (font (size 1.27 1.27)) hide)
     )
+    (property "Alternative" "" (at 92.71 175.895 0)
+      (effects (font (size 1.27 1.27)) hide)
+    )
     (pin "1")
     (pin "2")
@@
       (effects (font (size 1.27 1.27)) hide)
     )
+    (property "Alternative" "" (at 225.171 120.396 0)
+      (effects (font (size 1.27 1.27)) hide)
+    )
     (pin "1")
     (pin "2")
@@
     )
     (property "Mouser" "" (at 194.945 174.625 0)
+      (effects (font (size 1.27 1.27)) hide)
+    )
+    (property "Comment" "Use Original" (at 194.945 174.625 0)
+      (effects (font (size 1.27 1.27)) hide)
+    )
+    (property "Alternative" "" (at 194.945 174.625 0)
       (effects (font (size 1.27 1.27)) hide)
     )
@@
       (effects (font (size 1.27 1.27)) hide)
     )
+    (property "Comment" "Use Original" (at 244.221 121.666 0)
+      (effects (font (size 1.27 1.27)) hide)
+    )
+    (property "Alternative" "" (at 244.221 121.666 0)
+      (effects (font (size 1.27 1.27)) hide)
+    )
     (pin "1")
     (pin "2")
@@
       (effects (font (size 1.27 1.27)) hide)
     )
-    (property "Mouser" "" (at 261.366 85.471 0)
+    (property "Mouser" "815-AB-3.579545-B2" (at 261.366 85.471 0)
+      (effects (font (size 1.27 1.27)) hide)
+    )
+    (property "Alternative" "" (at 261.366 85.471 0)
       (effects (font (size 1.27 1.27)) hide)
     )
@@
       (effects (font (size 1.27 1.27)) hide)
     )
-    (property "Mouser" "" (at 222.885 155.575 0)
+    (property "Mouser" "71-CMF5010R000FHEK" (at 222.885 155.575 0)
+      (effects (font (size 1.27 1.27)) hide)
+    )
+    (property "Alternative" "" (at 222.885 155.575 0)
       (effects (font (size 1.27 1.27)) hide)
     )
@@
       (effects (font (size 1.27 1.27)) hide)
     )
-    (property "Mouser" "" (at 111.76 97.79 0)
+    (property "Mouser" "71-RN60E1003F" (at 111.76 97.79 0)
+      (effects (font (size 1.27 1.27)) hide)
+    )
+    (property "Alternative" "" (at 111.76 97.79 0)
       (effects (font (size 1.27 1.27)) hide)
     )
@@
       (effects (font (size 1.27 1.27)) hide)
     )
+    (property "Alternative" "" (at 121.285 92.71 0)
+      (effects (font (size 1.27 1.27)) hide)
+    )
     (pin "1")
     (pin "2")
@@
       (effects (font (size 1.27 1.27)) hide)
     )
+    (property "Alternative" "" (at 105.41 92.71 0)
+      (effects (font (size 1.27 1.27)) hide)
+    )
+    (property "Comment" "Use Original" (at 105.41 92.71 0)
+      (effects (font (size 1.27 1.27)) hide)
+    )
     (pin "1")
     (pin "2")
@@
       (effects (font (size 1.27 1.27)) hide)
     )
-    (property "Mouser" "" (at 267.716 115.316 0)
+    (property "Mouser" "595-SN74HC04N" (at 267.716 115.316 0)
+      (effects (font (size 1.27 1.27)) hide)
+    )
+    (property "Alternative" "" (at 267.716 115.316 0)
       (effects (font (size 1.27 1.27)) hide)
     )
@@
       (effects (font (size 1.27 1.27)) hide)
     )
-    (property "Mouser" "" (at 144.78 123.825 0)
+    (property "Mouser" "595-SN74HC04N" (at 144.78 123.825 0)
+      (effects (font (size 1.27 1.27)) hide)
+    )
+    (property "Alternative" "" (at 144.78 123.825 0)
       (effects (font (size 1.27 1.27)) hide)
     )
@@
   )
   (symbol (lib_id "Connector:TestPoint") (at 167.64 173.355 0) (mirror x) (unit 1)
-    (in_bom yes) (on_board yes) (dnp no) (fields_autoplaced)
+    (in_bom no) (on_board yes) (dnp no) (fields_autoplaced)
     (property "Reference" "TP2" (at 165.1 175.3869 0)
       (effects (font (size 1.27 1.27)) (justify right))
@@
       (effects (font (size 1.27 1.27)) hide)
     )
+    (property "Alternative" "" (at 167.64 173.355 0)
+      (effects (font (size 1.27 1.27)) hide)
+    )
     (pin "1")
     (instances
@@
       (effects (font (size 1.27 1.27)) hide)
     )
+    (property "Alternative" "" (at 173.99 135.255 0)
+      (effects (font (size 1.27 1.27)) hide)
+    )
     (pin "1")
     (pin "2")
@@
       (effects (font (size 1.27 1.27)) hide)
     )
-    (property "Mouser" "" (at 143.51 113.665 0)
+    (property "Mouser" "71-RN60D-F-1M/R" (at 143.51 113.665 0)
+      (effects (font (size 1.27 1.27)) hide)
+    )
+    (property "Alternative" "" (at 143.51 113.665 0)
       (effects (font (size 1.27 1.27)) hide)
     )
@@
       (effects (font (size 1.27 1.27)) hide)
     )
+    (property "Alternative" "" (at 105.41 113.665 0)
+      (effects (font (size 1.27 1.27)) hide)
+    )
+    (property "Comment" "Use Original" (at 105.41 113.665 0)
+      (effects (font (size 1.27 1.27)) hide)
+    )
     (pin "1")
     (pin "2")
@@
       (effects (font (size 1.27 1.27)) hide)
     )
-    (property "Mouser" "" (at 222.885 163.83 0)
+    (property "Mouser" "71-RN60D2203F" (at 222.885 163.83 0)
+      (effects (font (size 1.27 1.27)) hide)
+    )
+    (property "Alternative" "" (at 222.885 163.83 0)
       (effects (font (size 1.27 1.27)) hide)
     )
@@
       (effects (font (size 1.27 1.27)) hide)
     )
+    (property "Alternative" "" (at 121.285 113.665 0)
+      (effects (font (size 1.27 1.27)) hide)
+    )
     (pin "1")
     (pin "2")
@@
       (effects (font (size 1.27 1.27)) hide)
     )
-    (property "Mouser" "" (at 186.055 123.825 0)
+    (property "Mouser" "595-SN74HC04N" (at 186.055 123.825 0)
+      (effects (font (size 1.27 1.27)) hide)
+    )
+    (property "Alternative" "" (at 186.055 123.825 0)
       (effects (font (size 1.27 1.27)) hide)
     )
@@
       (effects (font (size 1.27 1.27)) hide)
     )
+    (property "Alternative" "" (at 282.956 93.091 0)
+      (effects (font (size 1.27 1.27)) hide)
+    )
     (pin "1")
     (pin "2")
@@
       (effects (font (size 1.27 1.27)) hide)
     )
+    (property "Alternative" "" (at 236.22 165.735 0)
+      (effects (font (size 1.27 1.27)) hide)
+    )
     (pin "1")
     (pin "2")
@@
     )
     (property "Mouser" "810-FG28C0G1H060DNT6" (at 158.115 92.71 0)
+      (effects (font (size 1.27 1.27)) hide)
+    )
+    (property "Alternative" "" (at 158.115 92.71 0)
       (effects (font (size 1.27 1.27)) hide)
     )
@@
       (effects (font (size 1.27 1.27)) hide)
     )
+    (property "Alternative" "" (at 222.885 175.895 0)
+      (effects (font (size 1.27 1.27)) hide)
+    )
     (pin "1")
     (pin "2")
@@
   )
   (symbol (lib_id "Connector:TestPoint") (at 319.786 108.966 0) (unit 1)
-    (in_bom yes) (on_board yes) (dnp no) (fields_autoplaced)
+    (in_bom no) (on_board yes) (dnp no) (fields_autoplaced)
     (property "Reference" "TP1" (at 321.691 104.3939 0)
       (effects (font (size 1.27 1.27)) (justify left))
@@
       (effects (font (size 1.27 1.27)) hide)
     )
+    (property "Alternative" "" (at 319.786 108.966 0)
+      (effects (font (size 1.27 1.27)) hide)
+    )
     (pin "1")
     (instances
@@
       (effects (font (size 1.27 1.27)) hide)
     )
+    (property "Alternative" "" (at 282.956 123.571 0)
+      (effects (font (size 1.27 1.27)) hide)
+    )

Commit message: update before public
Parts:
- D3, D4: Alternative (none) -> LV2209
- R101, R102: Mouser 71-RN60E1003F -> (none)
- R68: Mouser 71-RN60E1002F -> (none)
- R70, R72: Mouser 71-RN60D-F-1M/R -> (none)
- R71: Mouser 71-CMF5010R000FHEK -> (none)
- R74: Mouser 71-RN60D2203F -> (none)
Changed lines of the file:
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@@
       (effects (font (size 1.27 1.27)) hide)
     )
-    (property "Mouser" "71-RN60E1002F" (at 191.135 173.355 0)
+    (property "Mouser" "" (at 191.135 173.355 0)
       (effects (font (size 1.27 1.27)) hide)
     )
@@
       (effects (font (size 1.27 1.27)) hide)
     )
-    (property "Mouser" "71-RN60D-F-1M/R" (at 260.096 100.711 0)
+    (property "Mouser" "" (at 260.096 100.711 0)
       (effects (font (size 1.27 1.27)) hide)
     )
@@
       (effects (font (size 1.27 1.27)) hide)
     )
-    (property "Mouser" "71-RN60E1003F" (at 111.76 108.585 0)
+    (property "Mouser" "" (at 111.76 108.585 0)
       (effects (font (size 1.27 1.27)) hide)
     )
@@
       (effects (font (size 1.27 1.27)) hide)
     )
-    (property "Mouser" "71-CMF5010R000FHEK" (at 222.885 155.575 0)
+    (property "Mouser" "" (at 222.885 155.575 0)
       (effects (font (size 1.27 1.27)) hide)
     )
@@
       (effects (font (size 1.27 1.27)) hide)
     )
-    (property "Mouser" "71-RN60E1003F" (at 111.76 97.79 0)
+    (property "Mouser" "" (at 111.76 97.79 0)
       (effects (font (size 1.27 1.27)) hide)
     )
@@
       (effects (font (size 1.27 1.27)) hide)
     )
-    (property "Alternative" "" (at 105.41 92.71 0)
+    (property "Alternative" "LV2209" (at 105.41 92.71 0)
       (effects (font (size 1.27 1.27)) hide)
     )
@@
       (effects (font (size 1.27 1.27)) hide)
     )
-    (property "Mouser" "71-RN60D-F-1M/R" (at 143.51 113.665 0)
+    (property "Mouser" "" (at 143.51 113.665 0)
       (effects (font (size 1.27 1.27)) hide)
     )
@@
       (effects (font (size 1.27 1.27)) hide)
     )
-    (property "Alternative" "" (at 105.41 113.665 0)
+    (property "Alternative" "LV2209" (at 105.41 113.665 0)
       (effects (font (size 1.27 1.27)) hide)
     )
@@
       (effects (font (size 1.27 1.27)) hide)
     )
-    (property "Mouser" "71-RN60D2203F" (at 222.885 163.83 0)
-      (effects (font (size 1.27 1.27)) hide)
-    )
+    (property "Mouser" "" (at 222.885 163.83 0)
+      (effects (font (size 1.27 1.27)) hide)
+    )

Commit message: More BOM Tweaks
Parts:
- R71: Mouser (none) -> 71-CMF5010R000FHEK
Changed lines of the file:
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@@
       (effects (font (size 1.27 1.27)) hide)
     )
-    (property "Mouser" "" (at 222.885 155.575 0)
+    (property "Mouser" "71-CMF5010R000FHEK" (at 222.885 155.575 0)
       (effects (font (size 1.27 1.27)) hide)
     )
