File: sheets/power.kicad_sch (KiCad schematic)
At the start: 73 parts, among them SW2 FCC-0001SW, T1 COIL, U11 74LS05, U12 74LS06, U28 PC4741, U29 PC4741, U33 74AS04, U37 LM2576T-5, U38 74HC32, U8 74HC04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

Commit message: Power Circuit Update 1
Parts:
- added Q?: A1442, symbol Device:Q_PNP_BCE
- added Q?: A1015, Package_TO_SOT_THT:TO-92_Inline, symbol Transistor_BJT:2SA1015
- added Q?: 2SC1815, Package_TO_SOT_THT:TO-92_Inline, symbol Transistor_BJT:2SC1815
- added R77: 10K, symbol Device:R_Small
- added R78: 1K, symbol Device:R_Small
- added R79: 510, symbol Device:R_Small
- added SW2: ~, symbol Switch:SW_Push_SPDT
Connections:
- net VCC: now also Q?.2 (C)
- net at C46.1, R67.1, U37.1 (VIN): no longer D1.2 (A)
- net at C44.2, T1.2 (AB): now also SW2.1 (A); no longer D1.1 (K)
- new net: Q?.3 (B), Q?.3 (E), R77.1
- new net: D1.1 (K), Q?.1 (E), R77.2, SW2.2 (B)
- new net: Q?.2 (C), R79.2
- new net: Q?.1 (E), R78.2
- new net: Q?.2 (C), R79.1
- new net: D1.2 (A), R78.1
- no-connect marks 10 -> 11
Other:
- moved on the sheet: C46, C47, D1, D2, L3, R67, SW2, U37

Commit message: Update Power Circuit 2
Parts:
- Q11: renamed from Q?; value 2SC1815 -> C1815
- Q12: renamed from Q?; footprint Package_TO_SOT_THT:TO-92_Inline -> Package_TO_SOT_THT:TO-92_Inline_Wide
- Q13: renamed from Q?; footprint (none) -> Package_TO_SOT_THT:TO-3P-3_Vertical
- R77, R78, R79: footprint (none) -> 1_NeoGeoLibrary:CAP3-5mm
Changed lines of the file:
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@@
   (junction (at 28.702 146.685) (diameter 0) (color 0 0 0 0)
-  )
-  (junction (at 73.406 81.026) (diameter 0) (color 0 0 0 0)
   )
   (junction (at 99.695 127) (diameter 0) (color 0 0 0 0)
@@
     (stroke (width 0) (type default) (color 0 0 0 0))
   )
-  (wire (pts (xy 36.83 98.298) (xy 45.212 98.298))
-    (stroke (width 0) (type default) (color 0 0 0 0))
-  )
   (wire (pts (xy 48.895 132.08) (xy 59.055 132.08))
     (stroke (width 0) (type default) (color 0 0 0 0))
@@
   )
   (wire (pts (xy 42.926 67.31) (xy 51.562 67.31))
-    (stroke (width 0) (type default) (color 0 0 0 0))
-  )
-  (wire (pts (xy 73.406 81.026) (xy 73.406 91.694))
     (stroke (width 0) (type default) (color 0 0 0 0))
   )
@@
   (symbol (lib_id "Device:Q_PNP_BCE") (at 92.202 77.47 180) (unit 1)
     (in_bom yes) (on_board yes) (fields_autoplaced)
-    (property "Reference" "Q?" (id 0) (at 86.36 76.1999 0)
+    (property "Reference" "Q13" (id 0) (at 86.36 76.1999 0)
       (effects (font (size 1.27 1.27)) (justify left))
     )
@@
       (effects (font (size 1.27 1.27)) (justify left))
     )
-    (property "Footprint" "" (id 2) (at 87.122 80.01 0)
+    (property "Footprint" "Package_TO_SOT_THT:TO-3P-3_Vertical" (id 2) (at 87.122 80.01 0)
       (effects (font (size 1.27 1.27)) hide)
     )
@@
   (symbol (lib_id "Transistor_BJT:2SA1015") (at 75.946 72.39 180) (unit 1)
     (in_bom yes) (on_board yes) (fields_autoplaced)
-    (property "Reference" "Q?" (id 0) (at 69.85 71.1199 0)
+    (property "Reference" "Q12" (id 0) (at 69.85 71.1199 0)
       (effects (font (size 1.27 1.27)) (justify left))
     )
@@
       (effects (font (size 1.27 1.27)) (justify left))
     )
-    (property "Footprint" "Package_TO_SOT_THT:TO-92_Inline" (id 2) (at 70.866 70.485 0)
+    (property "Footprint" "Package_TO_SOT_THT:TO-92_Inline_Wide" (id 2) (at 70.866 70.485 0)
       (effects (font (size 1.27 1.27) italic) (justify left) hide)
     )
@@
   (symbol (lib_id "Transistor_BJT:2SC1815") (at 56.642 96.012 270) (mirror x) (unit 1)
     (in_bom yes) (on_board yes) (fields_autoplaced)
-    (property "Reference" "Q?" (id 0) (at 56.642 86.36 90))
-    (property "Value" "2SC1815" (id 1) (at 56.642 88.9 90))
+    (property "Reference" "Q11" (id 0) (at 56.642 86.36 90))
+    (property "Value" "C1815" (id 1) (at 56.642 88.9 90))
     (property "Footprint" "Package_TO_SOT_THT:TO-92_Inline" (id 2) (at 54.737 90.932 0)
       (effects (font (size 1.27 1.27) italic) (justify left) hide)
@@
     (property "Reference" "R78" (id 0) (at 47.498 82.296 90))
     (property "Value" "1K" (id 1) (at 49.784 82.296 90))
-    (property "Footprint" "" (id 2) (at 51.562 82.296 0)
+    (property "Footprint" "1_NeoGeoLibrary:CAP3-5mm" (id 2) (at 51.562 82.296 0)
       (effects (font (size 1.27 1.27)) hide)
     )
@@
     (property "Reference" "R77" (id 0) (at 70.612 57.912 90))
     (property "Value" "10K" (id 1) (at 70.612 60.198 90))
-    (property "Footprint" "" (id 2) (at 70.612 61.976 0)
+    (property "Footprint" "1_NeoGeoLibrary:CAP3-5mm" (id 2) (at 70.612 61.976 0)
       (effects (font (size 1.27 1.27)) hide)
     )
@@
     (property "Reference" "R79" (id 0) (at 67.564 76.962 90))
     (property "Value" "510" (id 1) (at 67.564 79.248 90))
-    (property "Footprint" "" (id 2) (at 67.564 81.026 0)
-      (effects (font (size 1.27 1.27)) hide)
-    )
+    (property "Footprint" "1_NeoGeoLibrary:CAP3-5mm" (id 2) (at 67.564 81.026 0)
+      (effects (font (size 1.27 1.27)) hide)
+    )

Commit message: Update Power Circuit 3
Parts:
- removed SW2: FCC-0001SW, Button_Switch_THT:SW_Tactile_Straight_KSL0Axx1LFTR, symbol Switch:SW_SPST
Connections:
- net GND: now also R67.2, U37.5 (~{ON}/OFF)
- no-connect marks 11 -> 13
Changed lines of the file:
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@@
   (no_connect (at 351.79 221.996))
   (no_connect (at 38.1 187.96))
+  (no_connect (at 97.282 77.47))
+  (no_connect (at 56.642 101.092))
   (no_connect (at 366.268 229.87))
   (no_connect (at 38.1 172.72))
@@
     (stroke (width 0) (type default) (color 0 0 0 0))
   )
-  (wire (pts (xy 205.232 49.784) (xy 215.9 49.784))
+  (wire (pts (xy 195.072 49.784) (xy 215.9 49.784))
     (stroke (width 0) (type default) (color 0 0 0 0))
   )
@@
     (pin "1")
   )
-  (symbol (lib_id "Switch:SW_SPST") (at 200.152 49.784 0) (unit 1)
-    (in_bom yes) (on_board yes)
-    (property "Reference" "SW2" (id 0) (at 200.152 46.736 0))
-    (property "Value" "FCC-0001SW" (id 1) (at 200.152 52.832 0))
-    (property "Footprint" "Button_Switch_THT:SW_Tactile_Straight_KSL0Axx1LFTR" (id 2) (at 200.152 49.784 0)
-      (effects (font (size 1.27 1.27)) hide)
-    )
-    (property "Datasheet" "" (id 3) (at 200.152 49.784 0)
-      (effects (font (size 1.27 1.27)) hide)
-    )
-    (pin "1")
-    (pin "2")
-  )
   (symbol (lib_id "74xx:74LS04") (at 180.34 259.08 0) (unit 7)
     (in_bom yes) (on_board yes) (fields_autoplaced)
@@
   (symbol (lib_id "power:VCC") (at 89.662 82.55 180) (unit 1)
     (in_bom yes) (on_board yes)
-    (property "Reference" "#PWR?" (id 0) (at 89.662 78.74 0)
-      (effects (font (size 1.27 1.27)) hide)
-    )
+    (property "Reference" "#PWR0278" (id 0) (at 89.662 78.74 0)
+      (effects (font (size 1.27 1.27)) hide)
+    )

Commit message: Update Power Circuit 4
Parts:
- added D11, D12, D13: 1N41, symbol Device:D_Small
- added R80: 470, 1_NeoGeoLibrary:CAP3-5mm, symbol Device:R_Small
- added R81: 100, 1_NeoGeoLibrary:CAP3-5mm, symbol Device:R_Small
- added R82: 510, 1_NeoGeoLibrary:CAP3-5mm, symbol Device:R_Small
Connections:
- net GND: now also D12.1 (K)
- net at C46.1, R67.1, U37.1 (VIN): now also D1.2 (A)
- net at Q13.1 (B): now also Q12.2 (C)
- net at Q13.3 (E), R77.1: now also R81.1; no longer Q12.3 (B)
- net at Q12.1 (E), R77.2, SW2.2 (B): now also D13.2 (A); no longer D1.1 (K)
- net at R79.2: now also Q12.3 (B), R81.2, R82.2; no longer Q12.2 (C)
- net at Q11.3 (B): now also R80.2
- net at R78.1: now also D13.1 (K), R80.1; no longer D1.2 (A)
- new net: D11.1 (K), D12.2 (A)
- new net: D1.1 (K), D11.2 (A), R82.1
- no-connect marks 13 -> 11
Other:
- moved on the sheet: C46, C47, D1, D2, L3, Q11, Q12, Q13, R67, R77, R78, R79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

Commit message: Update Power Circuit 5
Parts:
- D11, D12, D13: footprint (none) -> Diode_THT:D_A-405_P10.16mm_Horizontal
Changed lines of the file:
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@@
       (effects (font (size 1.27 1.27)) (justify right))
     )
-    (property "Footprint" "" (id 2) (at 128.27 82.804 90)
+    (property "Footprint" "Diode_THT:D_A-405_P10.16mm_Horizontal" (id 2) (at 128.27 82.804 90)
       (effects (font (size 1.27 1.27)) hide)
     )
@@
       (effects (font (size 1.27 1.27)) (justify right))
     )
-    (property "Footprint" "" (id 2) (at 51.562 80.01 90)
+    (property "Footprint" "Diode_THT:D_A-405_P10.16mm_Horizontal" (id 2) (at 51.562 80.01 90)
       (effects (font (size 1.27 1.27)) hide)
     )
@@
       (effects (font (size 1.27 1.27)) (justify right))
     )
-    (property "Footprint" "" (id 2) (at 128.27 74.168 90)
-      (effects (font (size 1.27 1.27)) hide)
-    )
+    (property "Footprint" "Diode_THT:D_A-405_P10.16mm_Horizontal" (id 2) (at 128.27 74.168 90)
+      (effects (font (size 1.27 1.27)) hide)
+    )

Commit message: Power Circuit Update 6
Parts:
- SW2: footprint (none) -> Button_Switch_THT:SW_Slide_1P2T_CK_OS102011MS2Q
Connections:
- net at Q13.3 (E), R77.1, R81.1: now also D1.1 (K)
- net at Q12.3 (B), R79.2, R81.2: now also R82.1; no longer R82.2
- new net: D11.2 (A), R82.2
Other:
- moved on the sheet: C46, C47, D1, D11, D12, D13, D2, L3, Q11, Q12, Q13, R67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

Commit message: Update Power Circuit 7
Connections:
- net at Q13.3 (E), R77.1, R81.1: no longer D1.1 (K)
- net at D13.2 (A), Q12.1 (E), R77.2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: now also D1.1 (K)
Other:
- moved on the sheet: C46, C47, D1, D2, L3, R67, U37

Commit message: Update Power Circuit 8
Connections:
- net at C46.1, D1.2 (A), R67.1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: now also D11.2 (A), R82.2
Changed lines of the file:
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@@
   (junction (at 140.462 141.605) (diameter 0) (color 0 0 0 0)
   )
+  (junction (at 133.858 60.706) (diameter 0) (color 0 0 0 0)
+  )
   (junction (at 152.146 246.38) (diameter 0) (color 0 0 0 0)
   )
@@
   )
   (junction (at 22.86 187.96) (diameter 0) (color 0 0 0 0)
+  )
+  (junction (at 108.966 94.234) (diameter 0) (color 0 0 0 0)
   )
   (junction (at 140.589 60.706) (diameter 0) (color 0 0 0 0)
@@
     (stroke (width 0) (type default) (color 0 0 0 0))
   )
+  (wire (pts (xy 133.858 60.706) (xy 133.858 94.234))
+    (stroke (width 0) (type default) (color 0 0 0 0))
+  )
   (wire (pts (xy 130.175 132.08) (xy 140.335 132.08))
     (stroke (width 0) (type default) (color 0 0 0 0))
@@
     (stroke (width 0) (type default) (color 0 0 0 0))
   )
+  (wire (pts (xy 108.966 94.234) (xy 108.966 94.996))
+    (stroke (width 0) (type default) (color 0 0 0 0))
+  )
   (wire (pts (xy 152.146 246.38) (xy 180.34 246.38))
     (stroke (width 0) (type default) (color 0 0 0 0))
@@
     (stroke (width 0) (type default) (color 0 0 0 0))
   )
-  (wire (pts (xy 129.921 60.706) (xy 140.589 60.706))
+  (wire (pts (xy 129.921 60.706) (xy 133.858 60.706))
     (stroke (width 0) (type default) (color 0 0 0 0))
   )
@@
     (stroke (width 0) (type default) (color 0 0 0 0))
   )
+  (wire (pts (xy 133.858 60.706) (xy 140.589 60.706))
+    (stroke (width 0) (type default) (color 0 0 0 0))
+  )
   (wire (pts (xy 191.135 132.08) (xy 201.295 132.08))
     (stroke (width 0) (type default) (color 0 0 0 0))
@@
     (stroke (width 0) (type default) (color 0 0 0 0))
   )
-  (wire (pts (xy 108.966 93.599) (xy 108.966 94.996))
+  (wire (pts (xy 108.966 93.599) (xy 108.966 94.234))
     (stroke (width 0) (type default) (color 0 0 0 0))
   )
@@
     (stroke (width 0) (type default) (color 0 0 0 0))
   )
+  (wire (pts (xy 108.966 94.234) (xy 133.858 94.234))
+    (stroke (width 0) (type default) (color 0 0 0 0))
+  )
