File: sheets/video.kicad_sch (KiCad schematic)
At the start: 28 parts, among them U10 74LS273, U11 74LS05, U5 NEO-G0, U6 uPD4364CX-12, U7 uPD4364CX-12, U8 74HC04, U9 74LS273

Commit message: Merged in schematics from stable with footprints
Parts:
- U10, U9: footprint (none) -> Package_DIP:DIP-20_W7.62mm
- U11, U8: footprint (none) -> Package_DIP:DIP-14_W7.62mm
- U5: footprint (none) -> Package_LCC:PLCC-84

Commit message: FIX 74AS04 and 74HC04
Parts:
- renumbered U8 to U80
Changed lines of the file:
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@@
   (symbol (lib_id "74xx:74HC04") (at 93.726 202.184 0) (unit 5)
     (in_bom yes) (on_board yes) (fields_autoplaced)
-    (property "Reference" "U8" (id 0) (at 93.726 193.548 0))
-    (property "Value" "74HC04" (id 1) (at 93.726 196.088 0))
+    (property "Reference" "U80" (id 0) (at 93.726 193.04 0))
+    (property "Value" "74HC04" (id 1) (at 93.726 195.58 0))
     (property "Footprint" "Package_DIP:DIP-14_W7.62mm" (id 2) (at 93.726 202.184 0)
       (effects (font (size 1.27 1.27)) hide)
@@
   (symbol (lib_id "74xx:74HC04") (at 69.342 202.184 0) (unit 6)
     (in_bom yes) (on_board yes) (fields_autoplaced)
-    (property "Reference" "U8" (id 0) (at 69.342 193.548 0))
-    (property "Value" "74HC04" (id 1) (at 69.342 196.088 0))
+    (property "Reference" "U80" (id 0) (at 69.342 193.04 0))
+    (property "Value" "74HC04" (id 1) (at 69.342 195.58 0))
     (property "Footprint" "Package_DIP:DIP-14_W7.62mm" (id 2) (at 69.342 202.184 0)
       (effects (font (size 1.27 1.27)) hide)

Commit message: Sync footprints from Nightly Build
Parts:
- U5: footprint Package_LCC:PLCC-84 -> 1_NeoGeoLibrary:NEO-G0
- U6, U7: footprint Package_DIP:DIP-28_W15.24mm -> Package_DIP:DIP-28_W7.62mm
Changed lines of the file:
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@@
     (property "Reference" "U6" (id 0) (at 170.434 94.234 0))
     (property "Value" "uPD4364CX-12" (id 1) (at 177.038 137.414 0))
-    (property "Footprint" "Package_DIP:DIP-28_W15.24mm" (id 2) (at 177.038 120.65 0)
+    (property "Footprint" "Package_DIP:DIP-28_W7.62mm" (id 2) (at 177.038 120.65 0)
       (effects (font (size 1.27 1.27)) hide)
     )
@@
     (property "Reference" "U5" (id 0) (at 130.81 155.448 0))
     (property "Value" "NEO-G0" (id 1) (at 139.7 247.142 0))
-    (property "Footprint" "Package_LCC:PLCC-84" (id 2) (at 139.7 214.884 0)
+    (property "Footprint" "1_NeoGeoLibrary:NEO-G0" (id 2) (at 139.7 214.884 0)
       (effects (font (size 1.27 1.27)) hide)
     )
@@
     (property "Reference" "U7" (id 0) (at 170.434 39.878 0))
     (property "Value" "uPD4364CX-12" (id 1) (at 177.038 83.058 0))
-    (property "Footprint" "Package_DIP:DIP-28_W15.24mm" (id 2) (at 177.038 66.294 0)
+    (property "Footprint" "Package_DIP:DIP-28_W7.62mm" (id 2) (at 177.038 66.294 0)
       (effects (font (size 1.27 1.27)) hide)
     )

Commit message: Fix U8 Unused pins to GND and NC Added C67 to A12 Pin 2 of U6
Parts:
- added C67: 220pF, 1_NeoGeoLibrary:CAP3-5mm, symbol Device:C_Small
Connections:
- net GND: now also C67.1
- net PALBNK: now also C67.2
Changed lines of the file:
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@@
   (junction (at 293.37 167.386) (diameter 0) (color 0 0 0 0)
+  )
+  (junction (at 141.478 128.27) (diameter 0) (color 0 0 0 0)
   )
   (junction (at 162.052 86.614) (diameter 0) (color 0 0 0 0)
@@
     (pin "1")
     (pin "2")
+  )
+  (symbol (lib_id "power:GND") (at 141.478 133.35 0) (unit 1)
+    (in_bom yes) (on_board yes) (fields_autoplaced)
+    (property "Reference" "#PWR0274" (id 0) (at 141.478 139.7 0)
+      (effects (font (size 1.27 1.27)) hide)
+    )
+    (property "Value" "GND" (id 1) (at 141.478 138.43 0))
+    (property "Footprint" "" (id 2) (at 141.478 133.35 0)
+      (effects (font (size 1.27 1.27)) hide)
+    )
+    (property "Datasheet" "" (id 3) (at 141.478 133.35 0)
+      (effects (font (size 1.27 1.27)) hide)
+    )
+    (pin "1")
   )
   (symbol (lib_id "Device:R_Small") (at 300.482 118.11 270) (mirror x) (unit 1)
@@
       (effects (font (size 1.27 1.27)) hide)
     )
+    (pin "1")
+    (pin "2")
+  )
+  (symbol (lib_id "Device:C_Small") (at 141.478 130.81 180) (unit 1)
+    (in_bom yes) (on_board yes)
+    (property "Reference" "C67" (id 0) (at 144.018 130.175 0)
+      (effects (font (size 1.27 1.27)) (justify right))
+    )
+    (property "Value" "220pF" (id 1) (at 144.018 132.08 0)
+      (effects (font (size 1.27 1.27)) (justify right))
+    )
+    (property "Footprint" "1_NeoGeoLibrary:CAP3-5mm" (id 2) (at 141.478 130.81 0)
+      (effects (font (size 1.27 1.27)) hide)
+    )
+    (property "Datasheet" "" (id 3) (at 141.478 130.81 0)
+      (effects (font (size 1.27 1.27)) hide)
+    )

Commit message: Schematics Footprint updates
Parts:
- U10, U9: footprint Package_DIP:DIP-20_W7.62mm -> 1_NeoGeoLibrary:DIP-20_W7.62mm
- U11, U80: footprint Package_DIP:DIP-14_W7.62mm -> 1_NeoGeoLibrary:DIP-14_W7.62mm
- U6, U7: footprint Package_DIP:DIP-28_W7.62mm -> 1_NeoGeoLibrary:DIP-28_W7.62mm
Changed lines of the file:
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@@
       (effects (font (size 1.27 1.27)) (justify left))
     )
-    (property "Footprint" "Package_DIP:DIP-20_W7.62mm" (at 238.506 146.558 0)
+    (property "Footprint" "1_NeoGeoLibrary:DIP-20_W7.62mm" (at 238.506 146.558 0)
       (effects (font (size 1.27 1.27)) hide)
     )
@@
       (effects (font (size 1.27 1.27)))
     )
-    (property "Footprint" "Package_DIP:DIP-14_W7.62mm" (at 282.194 177.038 0)
+    (property "Footprint" "1_NeoGeoLibrary:DIP-14_W7.62mm" (at 282.194 177.038 0)
       (effects (font (size 1.27 1.27)) hide)
     )
@@
       (effects (font (size 1.27 1.27)))
     )
-    (property "Footprint" "Package_DIP:DIP-14_W7.62mm" (at 93.726 202.184 0)
+    (property "Footprint" "1_NeoGeoLibrary:DIP-14_W7.62mm" (at 93.726 202.184 0)
       (effects (font (size 1.27 1.27)) hide)
     )
@@
       (effects (font (size 1.27 1.27)) (justify left))
     )
-    (property "Footprint" "Package_DIP:DIP-20_W7.62mm" (at 238.506 73.914 0)
+    (property "Footprint" "1_NeoGeoLibrary:DIP-20_W7.62mm" (at 238.506 73.914 0)
       (effects (font (size 1.27 1.27)) hide)
     )
@@
       (effects (font (size 1.27 1.27)))
     )
-    (property "Footprint" "Package_DIP:DIP-28_W7.62mm" (at 177.038 120.65 0)
+    (property "Footprint" "1_NeoGeoLibrary:DIP-28_W7.62mm" (at 177.038 120.65 0)
       (effects (font (size 1.27 1.27)) hide)
     )
@@
       (effects (font (size 1.27 1.27)))
     )
-    (property "Footprint" "Package_DIP:DIP-28_W7.62mm" (at 177.038 66.294 0)
+    (property "Footprint" "1_NeoGeoLibrary:DIP-28_W7.62mm" (at 177.038 66.294 0)
       (effects (font (size 1.27 1.27)) hide)
     )
@@
       (effects (font (size 1.27 1.27)))
     )
-    (property "Footprint" "Package_DIP:DIP-14_W7.62mm" (at 259.842 213.36 0)
+    (property "Footprint" "1_NeoGeoLibrary:DIP-14_W7.62mm" (at 259.842 213.36 0)
       (effects (font (size 1.27 1.27)) hide)
     )
@@
       (effects (font (size 1.27 1.27)))
     )
-    (property "Footprint" "Package_DIP:DIP-14_W7.62mm" (at 69.342 202.184 0)
+    (property "Footprint" "1_NeoGeoLibrary:DIP-14_W7.62mm" (at 69.342 202.184 0)
       (effects (font (size 1.27 1.27)) hide)
     )
@@
       (effects (font (size 1.27 1.27)))
     )
-    (property "Footprint" "Package_DIP:DIP-14_W7.62mm" (at 282.194 130.81 0)
+    (property "Footprint" "1_NeoGeoLibrary:DIP-14_W7.62mm" (at 282.194 130.81 0)
       (effects (font (size 1.27 1.27)) hide)
     )
@@
       (effects (font (size 1.27 1.27)))
     )
-    (property "Footprint" "Package_DIP:DIP-14_W7.62mm" (at 272.796 83.312 0)
+    (property "Footprint" "1_NeoGeoLibrary:DIP-14_W7.62mm" (at 272.796 83.312 0)
       (effects (font (size 1.27 1.27)) hide)
     )
@@
       (effects (font (size 1.27 1.27)))
     )
-    (property "Footprint" "Package_DIP:DIP-14_W7.62mm" (at 259.842 227.076 0)
+    (property "Footprint" "1_NeoGeoLibrary:DIP-14_W7.62mm" (at 259.842 227.076 0)
       (effects (font (size 1.27 1.27)) hide)
     )
@@
       (effects (font (size 1.27 1.27)))
     )
-    (property "Footprint" "Package_DIP:DIP-14_W7.62mm" (at 259.842 199.644 0)
-      (effects (font (size 1.27 1.27)) hide)
-    )
+    (property "Footprint" "1_NeoGeoLibrary:DIP-14_W7.62mm" (at 259.842 199.644 0)
+      (effects (font (size 1.27 1.27)) hide)
+    )

Commit message: Some tweaks
Other:
- company: (none) -> SNK
- title: (none) -> NeoGeo AES
Changed lines of the file:
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@@
 (kicad_sch (version 20230121) (generator eeschema)
   (paper "A3")
+  (title_block
+    (title "NeoGeo AES")
+    (date "2023-08-19")
+    (rev "3.5")
+    (company "SNK")
+    (comment 3 "https://github.com/Board-Folk")
+    (comment 4 "Recreated By The Board Folk Team")
+  )
   (junction (at 293.37 71.882) (diameter 0) (color 0 0 0 0)
   )

Commit message: Updates to PCB Move P2 Joystick Port Move Memory Card Move Holes at top right Silkscreen added Update Titles
Other:
- title: NeoGeo AES -> NeoGeo AES 3-5
Changed lines of the file:
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@@
   (paper "A3")
   (title_block
-    (title "NeoGeo AES")
-    (date "2023-08-19")
-    (rev "3.5")
+    (title "NeoGeo AES 3-5")
+    (date "2023-08-27")
+    (rev "BF1.1")
     (company "SNK")
     (comment 3 "https://github.com/Board-Folk")
