File: sheets/video.kicad_sch (KiCad schematic)
At the start: 29 parts, among them U10 74LS273, U11 74LS05, U5 NEO-G0, U6 uPD4364CX-12, U7 uPD4364CX-12, U80 74HC04, U9 74LS273

Commit message: Update BF1.4
Update Mouser Parts
Update Silkscreen for Memory Slot
Update Silkscreen for BF1.4 Version and date
Generate Gerbers and BOM files
Parts:
- R1, R2, R3: Mouser 71-CMF501K0000FHEA -> 594-5063JD1K000FT
- R10, R14, R18: Mouser (none) -> 594-5063JD220R0F
- R11, R15, R7: Mouser (none) -> 594-5063JD3K900F
- R12, R16, R8: Mouser (none) -> 594-5063JD2K200FT
- R13, R17, R9: Mouser (none) -> 594-5063JD470R0FT
- R19, R20, R21: Mouser (none) -> 594-5063JD150R0FT
- R4, R5, R6: Mouser (none) -> 594-5063JD8K200FT
- U6, U7: Alternative (none) -> JEDEC 6264 (8k x 8) SRAM; Mouser (none) -> 972-5962-3829407MXA
Changed lines of the file:
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@@
   (title_block
     (title "NeoGeo AES 3-5")
-    (date "2023-12-30")
-    (rev "BF1.3")
+    (date "2024-01-06")
+    (rev "BF1.4")
     (company "SNK")
     (comment 3 "https://github.com/Board-Folk")
@@
       (effects (font (size 1.27 1.27)) hide)
     )
-    (property "Mouser" "" (at 286.258 74.93 0)
+    (property "Mouser" "594-5063JD220R0F" (at 286.258 74.93 0)
       (effects (font (size 1.27 1.27)) hide)
     )
@@
       (effects (font (size 1.27 1.27)) hide)
     )
-    (property "Mouser" "" (at 286.258 121.158 0)
+    (property "Mouser" "594-5063JD220R0F" (at 286.258 121.158 0)
       (effects (font (size 1.27 1.27)) hide)
     )
@@
       (effects (font (size 1.27 1.27)) hide)
     )
-    (property "Mouser" "" (at 300.482 71.882 0)
+    (property "Mouser" "594-5063JD150R0FT" (at 300.482 71.882 0)
       (effects (font (size 1.27 1.27)) hide)
     )
@@
       (effects (font (size 1.27 1.27)) hide)
     )
-    (property "Mouser" "" (at 286.258 50.546 0)
+    (property "Mouser" "594-5063JD3K900F" (at 286.258 50.546 0)
       (effects (font (size 1.27 1.27)) hide)
     )
@@
       (effects (font (size 1.27 1.27)) hide)
     )
-    (property "Mouser" "" (at 286.258 161.29 0)
+    (property "Mouser" "594-5063JD470R0FT" (at 286.258 161.29 0)
       (effects (font (size 1.27 1.27)) hide)
     )
@@
       (effects (font (size 1.27 1.27)) hide)
     )
-    (property "Mouser" "" (at 293.37 82.042 0)
+    (property "Mouser" "594-5063JD8K200FT" (at 293.37 82.042 0)
       (effects (font (size 1.27 1.27)) hide)
     )
@@
       (effects (font (size 1.27 1.27)) hide)
     )
-    (property "Mouser" "71-CMF501K0000FHEA" (at 286.258 62.738 0)
+    (property "Mouser" "594-5063JD1K000FT" (at 286.258 62.738 0)
       (effects (font (size 1.27 1.27)) hide)
     )
@@
       (effects (font (size 1.27 1.27)) hide)
     )
-    (property "Mouser" "" (at 300.482 118.11 0)
+    (property "Mouser" "594-5063JD150R0FT" (at 300.482 118.11 0)
       (effects (font (size 1.27 1.27)) hide)
     )
@@
       (effects (font (size 1.27 1.27)) hide)
     )
-    (property "Mouser" "" (at 286.258 143.002 0)
+    (property "Mouser" "594-5063JD3K900F" (at 286.258 143.002 0)
       (effects (font (size 1.27 1.27)) hide)
     )
@@
       (effects (font (size 1.27 1.27)) hide)
     )
-    (property "Mouser" "" (at 286.258 149.098 0)
+    (property "Mouser" "594-5063JD2K200FT" (at 286.258 149.098 0)
       (effects (font (size 1.27 1.27)) hide)
     )
@@
       (effects (font (size 1.27 1.27)) hide)
     )
-    (property "Mouser" "" (at 293.37 128.27 0)
+    (property "Mouser" "594-5063JD8K200FT" (at 293.37 128.27 0)
       (effects (font (size 1.27 1.27)) hide)
     )
@@
       (effects (font (size 1.27 1.27)) hide)
     )
-    (property "Mouser" "" (at 177.038 120.65 0)
+    (property "Mouser" "972-5962-3829407MXA" (at 177.038 120.65 0)
       (effects (font (size 1.27 1.27)) hide)
     )
-    (property "Alternative" "" (at 177.038 120.65 0)
+    (property "Alternative" "JEDEC 6264 (8k x 8) SRAM" (at 177.038 120.65 0)
       (effects (font (size 1.27 1.27)) hide)
     )
@@
       (effects (font (size 1.27 1.27)) hide)
     )
-    (property "Mouser" "" (at 177.038 66.294 0)
+    (property "Mouser" "972-5962-3829407MXA" (at 177.038 66.294 0)
       (effects (font (size 1.27 1.27)) hide)
     )
-    (property "Alternative" "" (at 177.038 66.294 0)
+    (property "Alternative" "JEDEC 6264 (8k x 8) SRAM" (at 177.038 66.294 0)
       (effects (font (size 1.27 1.27)) hide)
     )
@@
       (effects (font (size 1.27 1.27)) hide)
     )
-    (property "Mouser" "" (at 293.37 174.498 0)
+    (property "Mouser" "594-5063JD8K200FT" (at 293.37 174.498 0)
       (effects (font (size 1.27 1.27)) hide)
     )
@@
       (effects (font (size 1.27 1.27)) hide)
     )
-    (property "Mouser" "" (at 286.258 96.774 0)
+    (property "Mouser" "594-5063JD3K900F" (at 286.258 96.774 0)
       (effects (font (size 1.27 1.27)) hide)
     )
@@
       (effects (font (size 1.27 1.27)) hide)
     )
-    (property "Mouser" "" (at 286.258 115.062 0)
+    (property "Mouser" "594-5063JD470R0FT" (at 286.258 115.062 0)
       (effects (font (size 1.27 1.27)) hide)
     )
@@
       (effects (font (size 1.27 1.27)) hide)
     )
-    (property "Mouser" "" (at 300.482 164.338 0)
+    (property "Mouser" "594-5063JD150R0FT" (at 300.482 164.338 0)
       (effects (font (size 1.27 1.27)) hide)
     )
@@
       (effects (font (size 1.27 1.27)) hide)
     )
-    (property "Mouser" "" (at 286.258 167.386 0)
+    (property "Mouser" "594-5063JD220R0F" (at 286.258 167.386 0)
       (effects (font (size 1.27 1.27)) hide)
     )
@@
       (effects (font (size 1.27 1.27)) hide)
     )
-    (property "Mouser" "" (at 286.258 102.87 0)
+    (property "Mouser" "594-5063JD2K200FT" (at 286.258 102.87 0)
       (effects (font (size 1.27 1.27)) hide)
     )
@@
       (effects (font (size 1.27 1.27)) hide)
     )
-    (property "Mouser" "" (at 286.258 68.834 0)
+    (property "Mouser" "594-5063JD470R0FT" (at 286.258 68.834 0)
       (effects (font (size 1.27 1.27)) hide)
     )
@@
       (effects (font (size 1.27 1.27)) hide)
     )
-    (property "Mouser" "71-CMF501K0000FHEA" (at 286.258 155.194 0)
+    (property "Mouser" "594-5063JD1K000FT" (at 286.258 155.194 0)
       (effects (font (size 1.27 1.27)) hide)
     )
@@
       (effects (font (size 1.27 1.27)) hide)
     )
-    (property "Mouser" "" (at 286.258 56.642 0)
+    (property "Mouser" "594-5063JD2K200FT" (at 286.258 56.642 0)
       (effects (font (size 1.27 1.27)) hide)
     )
@@
       (effects (font (size 1.27 1.27)) hide)
     )
-    (property "Mouser" "71-CMF501K0000FHEA" (at 286.258 108.966 0)
+    (property "Mouser" "594-5063JD1K000FT" (at 286.258 108.966 0)
       (effects (font (size 1.27 1.27)) hide)
     )

Commit message: Update Silk
Update Ram Silk
Fix mouser wrong 6.8K
Update BOM, Gerbers ...
Parts:
- U6, U7: value uPD4364CX-12 -> 4364
Changed lines of the file:
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@@
       (effects (font (size 1.27 1.27)))
     )
-    (property "Value" "uPD4364CX-12" (at 177.038 137.414 0)
+    (property "Value" "4364" (at 177.038 137.414 0)
       (effects (font (size 1.27 1.27)))
     )
@@
       (effects (font (size 1.27 1.27)))
     )
-    (property "Value" "uPD4364CX-12" (at 177.038 83.058 0)
+    (property "Value" "4364" (at 177.038 83.058 0)
       (effects (font (size 1.27 1.27)))
     )

Commit message: Bom Updates
Parts:
- U6, U7: Mouser 972-5962-3829407MXA -> 913-AS7C164A-15PCN
Changed lines of the file:
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@@
       (effects (font (size 1.27 1.27)) hide)
     )
-    (property "Mouser" "972-5962-3829407MXA" (at 177.038 120.65 0)
+    (property "Mouser" "913-AS7C164A-15PCN" (at 177.038 120.65 0)
       (effects (font (size 1.27 1.27)) hide)
     )
@@
       (effects (font (size 1.27 1.27)) hide)
     )
-    (property "Mouser" "972-5962-3829407MXA" (at 177.038 66.294 0)
+    (property "Mouser" "913-AS7C164A-15PCN" (at 177.038 66.294 0)
       (effects (font (size 1.27 1.27)) hide)
     )
