File: sheets/card_interface.kicad_sch (KiCad schematic)
At the start: 3 parts, among them CN6 5535653-1, U38 74HC32, U8 74HC04

Commit message: Merged in schematics from stable with footprints
Parts:
- U38, U8: footprint (none) -> Package_DIP:DIP-14_W7.62mm

Commit message: FIX 74AS04 and 74HC04
Parts:
- renumbered U8 to U80
Changed lines of the file:
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@@
   (symbol (lib_id "74xx:74HC04") (at 121.285 143.51 0) (unit 3)
     (in_bom yes) (on_board yes) (fields_autoplaced)
-    (property "Reference" "U8" (id 0) (at 121.285 134.62 0))
+    (property "Reference" "U80" (id 0) (at 121.285 134.62 0))
     (property "Value" "74HC04" (id 1) (at 121.285 137.16 0))
     (property "Footprint" "Package_DIP:DIP-14_W7.62mm" (id 2) (at 121.285 143.51 0)

Commit message: Sync footprints from Nightly Build
Parts:
- CN6: footprint TE_5535653-1 -> 1_NeoGeoLibrary:CN6
Changed lines of the file:
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@@
     (property "Reference" "CN6" (id 0) (at 233.045 89.154 0))
     (property "Value" "5535653-1" (id 1) (at 233.045 91.694 0))
-    (property "Footprint" "TE_5535653-1" (id 2) (at 233.045 139.7 0)
+    (property "Footprint" "1_NeoGeoLibrary:CN6" (id 2) (at 233.045 139.7 0)
       (effects (font (size 1.27 1.27)) (justify bottom) hide)
     )

Commit message: Schematics Footprint updates
Parts:
- U38, U80: footprint Package_DIP:DIP-14_W7.62mm -> 1_NeoGeoLibrary:DIP-14_W7.62mm
Changed lines of the file:
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@@
       (effects (font (size 1.27 1.27)))
     )
-    (property "Footprint" "Package_DIP:DIP-14_W7.62mm" (at 140.335 129.54 0)
+    (property "Footprint" "1_NeoGeoLibrary:DIP-14_W7.62mm" (at 140.335 129.54 0)
       (effects (font (size 1.27 1.27)) hide)
     )
@@
       (effects (font (size 1.27 1.27)))
     )
-    (property "Footprint" "Package_DIP:DIP-14_W7.62mm" (at 164.465 161.29 0)
+    (property "Footprint" "1_NeoGeoLibrary:DIP-14_W7.62mm" (at 164.465 161.29 0)
       (effects (font (size 1.27 1.27)) hide)
     )
@@
       (effects (font (size 1.27 1.27)))
     )
-    (property "Footprint" "Package_DIP:DIP-14_W7.62mm" (at 121.285 143.51 0)
+    (property "Footprint" "1_NeoGeoLibrary:DIP-14_W7.62mm" (at 121.285 143.51 0)
       (effects (font (size 1.27 1.27)) hide)
     )
@@
       (effects (font (size 1.27 1.27)))
     )
-    (property "Footprint" "Package_DIP:DIP-14_W7.62mm" (at 170.815 132.08 0)
-      (effects (font (size 1.27 1.27)) hide)
-    )
+    (property "Footprint" "1_NeoGeoLibrary:DIP-14_W7.62mm" (at 170.815 132.08 0)
+      (effects (font (size 1.27 1.27)) hide)
+    )

Commit message: Some tweaks
Other:
- company: (none) -> SNK
- title: (none) -> NeoGeo AES
Changed lines of the file:
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@@
 (kicad_sch (version 20230121) (generator eeschema)
   (paper "A3")
+  (title_block
+    (title "NeoGeo AES")
+    (date "2023-08-19")
+    (rev "3.5")
+    (company "SNK")
+    (comment 3 "https://github.com/Board-Folk")
+    (comment 4 "Recreated By The Board Folk Team")
+  )
   (junction (at 202.565 75.565) (diameter 0) (color 0 0 0 0)
   )

Commit message: Updates to PCB Move P2 Joystick Port Move Memory Card Move Holes at top right Silkscreen added Update Titles
Other:
- title: NeoGeo AES -> NeoGeo AES 3-5
Changed lines of the file:
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@@
   (paper "A3")
   (title_block
-    (title "NeoGeo AES")
-    (date "2023-08-19")
-    (rev "3.5")
+    (title "NeoGeo AES 3-5")
+    (date "2023-08-27")
+    (rev "BF1.1")
     (company "SNK")
     (comment 3 "https://github.com/Board-Folk")
