File: sheets/card_interface.kicad_sch (KiCad schematic)
At the start: 3 parts, among them CN6 5535653-1, U38 74HC32, U80 74HC04

Commit message: More silkscreen tidy up, adding mouser components to BOM
Parts:
- CN6: Mouser (none) -> 571-5535653-1
Changed lines of the file:
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@@
       (effects (font (size 1.27 1.27)) (justify bottom) hide)
     )
-    (property "Mouser" "" (at 233.045 139.7 0)
+    (property "Mouser" "571-5535653-1" (at 233.045 139.7 0)
       (effects (font (size 1.27 1.27)) hide)
     )

Commit message: Little tweaks to silkscreen Updated BOM with mouser parts
Parts:
- CN6: Comment 5535653-1 -> (none)
- U38: Mouser (none) -> 595-SN74HC32N
- U80: Mouser (none) -> 595-SN74HC04N
Changed lines of the file:
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@@
     (title "NeoGeo AES 3-5")
     (date "2023-08-27")
-    (rev "BF1.1")
+    (rev "BF1.2")
     (company "SNK")
     (comment 3 "https://github.com/Board-Folk")
@@
       (effects (font (size 1.27 1.27)) hide)
     )
-    (property "Mouser" "" (at 140.335 129.54 0)
+    (property "Mouser" "595-SN74HC32N" (at 140.335 129.54 0)
+      (effects (font (size 1.27 1.27)) hide)
+    )
+    (property "Alternative" "" (at 140.335 129.54 0)
       (effects (font (size 1.27 1.27)) hide)
     )
@@
       (effects (font (size 1.27 1.27)) hide)
     )
-    (property "Comment" "5535653-1" (at 233.045 139.7 0)
+    (property "Comment" "" (at 233.045 139.7 0)
       (effects (font (size 1.27 1.27)) (justify bottom) hide)
     )
     (property "Mouser" "571-5535653-1" (at 233.045 139.7 0)
+      (effects (font (size 1.27 1.27)) hide)
+    )
+    (property "Alternative" "" (at 233.045 139.7 0)
       (effects (font (size 1.27 1.27)) hide)
     )
@@
       (effects (font (size 1.27 1.27)) hide)
     )
-    (property "Mouser" "" (at 164.465 161.29 0)
+    (property "Mouser" "595-SN74HC32N" (at 164.465 161.29 0)
+      (effects (font (size 1.27 1.27)) hide)
+    )
+    (property "Alternative" "" (at 164.465 161.29 0)
       (effects (font (size 1.27 1.27)) hide)
     )
@@
       (effects (font (size 1.27 1.27)) hide)
     )
-    (property "Mouser" "" (at 121.285 143.51 0)
+    (property "Mouser" "595-SN74HC04N" (at 121.285 143.51 0)
+      (effects (font (size 1.27 1.27)) hide)
+    )
+    (property "Alternative" "" (at 121.285 143.51 0)
       (effects (font (size 1.27 1.27)) hide)
     )
@@
       (effects (font (size 1.27 1.27)) hide)
     )
-    (property "Mouser" "" (at 170.815 132.08 0)
-      (effects (font (size 1.27 1.27)) hide)
-    )
+    (property "Mouser" "595-SN74HC32N" (at 170.815 132.08 0)
+      (effects (font (size 1.27 1.27)) hide)
+    )
+    (property "Alternative" "" (at 170.815 132.08 0)
+      (effects (font (size 1.27 1.27)) hide)
+    )

Commit message: update before public
Changed lines of the file:
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@@
     (stroke (width 0) (type default))
   )
-  (wire (pts (xy 188.595 173.355) (xy 188.595 180.34))
+  (wire (pts (xy 188.595 173.355) (xy 188.595 181.737))
     (stroke (width 0) (type default))
   )
@@
     (stroke (width 0) (type default))
   )
+  (wire (pts (xy 222.885 180.34) (xy 210.693 180.34))
+    (stroke (width 0) (type default))
+  )
   (wire (pts (xy 216.535 82.55) (xy 216.535 96.52))
     (stroke (width 0) (type default))
@@
   )
   (bus (pts (xy 202.565 75.565) (xy 263.525 75.565))
+    (stroke (width 0) (type default))
+  )
+  (wire (pts (xy 210.693 180.34) (xy 210.693 181.737))
     (stroke (width 0) (type default))
   )
@@
   )
   (wire (pts (xy 257.175 106.68) (xy 243.205 106.68))
+    (stroke (width 0) (type default))
+  )
+  (wire (pts (xy 210.693 181.737) (xy 188.595 181.737))
     (stroke (width 0) (type default))
   )
@@
     (stroke (width 0) (type default))
   )
-  (wire (pts (xy 188.595 180.34) (xy 206.375 180.34))
-    (stroke (width 0) (type default))
-  )
   (wire (pts (xy 222.885 137.16) (xy 194.945 137.16))
     (stroke (width 0) (type default))
@@
     (stroke (width 0) (type default))
   )
-  (wire (pts (xy 206.375 180.34) (xy 222.885 180.34))
-    (stroke (width 0) (type default))
-  )
