File: sheets/card_interface.kicad_sch (KiCad schematic)
At the start: 3 parts, among them CN6 5535653-1, U38 74HC32, U80 74HC04

Commit message: Update BF1.4
Update Mouser Parts
Update Silkscreen for Memory Slot
Update Silkscreen for BF1.4 Version and date
Generate Gerbers and BOM files
Parts:
- CN6: value 5535653-1 -> Memory Card Interface; Comment (none) -> Use Original; Mouser 571-5535653-1 -> (none)
Changed lines of the file:
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@@
   (title_block
     (title "NeoGeo AES 3-5")
-    (date "2023-12-30")
-    (rev "BF1.3")
+    (date "2024-01-06")
+    (rev "BF1.4")
     (company "SNK")
     (comment 3 "https://github.com/Board-Folk")
@@
       (effects (font (size 1.27 1.27)))
     )
-    (property "Value" "5535653-1" (at 233.045 91.694 0)
+    (property "Value" "Memory Card Interface" (at 233.045 91.694 0)
       (effects (font (size 1.27 1.27)))
     )
@@
       (effects (font (size 1.27 1.27)) hide)
     )
-    (property "Comment" "" (at 233.045 139.7 0)
+    (property "Comment" "Use Original" (at 233.045 139.7 0)
       (effects (font (size 1.27 1.27)) (justify bottom) hide)
     )
-    (property "Mouser" "571-5535653-1" (at 233.045 139.7 0)
-      (effects (font (size 1.27 1.27)) hide)
-    )
+    (property "Mouser" "" (at 233.045 139.7 0)
+      (effects (font (size 1.27 1.27)) hide)
+    )
