File: sheets/card_interface.kicad_sch (KiCad schematic)
At the start: 3 parts, among them CN6 Memory Card Interface, U38 74HC32, U80 74HC04

Commit message: Updated to Kicad 10
Other:
- moved on the sheet: CN6, U38A, U38B, U38C, U80C
