File: sheets/cartridge_slots.kicad_sch (KiCad schematic)
At the start: 3 parts, among them CN4 AXC90020, CN5 AXC90020, U33 74AS04

Commit message: Updates to PCB Move P2 Joystick Port Move Memory Card Move Holes at top right Silkscreen added Update Titles
Other:
- title: NeoGeo AES -> NeoGeo AES 3-5
Changed lines of the file:
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@@
   (paper "A3")
   (title_block
-    (title "NeoGeo AES")
-    (date "2023-08-19")
-    (rev "3.5")
+    (title "NeoGeo AES 3-5")
+    (date "2023-08-27")
+    (rev "BF1.1")
     (company "SNK")
     (comment 3 "https://github.com/Board-Folk")

Commit message: More silkscreen tidy up, adding mouser components to BOM
Parts:
- CN4, CN5: Mouser (none) -> 587-395-100-524-204
Changed lines of the file:
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@@
       (effects (font (size 1.27 1.27)) hide)
     )
-    (property "Mouser" "" (at 276.86 118.11 0)
+    (property "Mouser" "587-395-100-524-204" (at 276.86 118.11 0)
       (effects (font (size 1.27 1.27)) hide)
     )
@@
       (effects (font (size 1.27 1.27)) hide)
     )
-    (property "Mouser" "" (at 157.48 116.84 0)
+    (property "Mouser" "587-395-100-524-204" (at 157.48 116.84 0)
       (effects (font (size 1.27 1.27)) hide)
     )

Commit message: Little tweaks to silkscreen Updated BOM with mouser parts
Parts:
- U33: Mouser (none) -> 595-SN74AS04N
Changed lines of the file:
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@@
     (title "NeoGeo AES 3-5")
     (date "2023-08-27")
-    (rev "BF1.1")
+    (rev "BF1.2")
     (company "SNK")
     (comment 3 "https://github.com/Board-Folk")
@@
       (effects (font (size 1.27 1.27)) hide)
     )
-    (property "Mouser" "" (at 129.54 205.74 0)
+    (property "Mouser" "595-SN74AS04N" (at 129.54 205.74 0)
+      (effects (font (size 1.27 1.27)) hide)
+    )
+    (property "Alternative" "" (at 129.54 205.74 0)
       (effects (font (size 1.27 1.27)) hide)
     )
@@
       (effects (font (size 1.27 1.27)) hide)
     )
-    (property "Mouser" "" (at 114.3 205.74 0)
+    (property "Mouser" "595-SN74AS04N" (at 114.3 205.74 0)
+      (effects (font (size 1.27 1.27)) hide)
+    )
+    (property "Alternative" "" (at 114.3 205.74 0)
       (effects (font (size 1.27 1.27)) hide)
     )
@@
       (effects (font (size 1.27 1.27)) hide)
     )
+    (property "Alternative" "" (at 276.86 118.11 0)
+      (effects (font (size 1.27 1.27)) hide)
+    )
     (pin "a1")
     (pin "a10")
@@
       (effects (font (size 1.27 1.27)) hide)
     )
-    (property "Mouser" "" (at 93.472 85.09 0)
+    (property "Mouser" "595-SN74AS04N" (at 93.472 85.09 0)
+      (effects (font (size 1.27 1.27)) hide)
+    )
+    (property "Alternative" "" (at 93.472 85.09 0)
       (effects (font (size 1.27 1.27)) hide)
     )
@@
       (effects (font (size 1.27 1.27)) hide)
     )
+    (property "Alternative" "" (at 157.48 116.84 0)
+      (effects (font (size 1.27 1.27)) hide)
+    )
     (pin "a1")
     (pin "a10")
@@
       (effects (font (size 1.27 1.27)) hide)
     )
-    (property "Mouser" "" (at 242.57 203.2 0)
+    (property "Mouser" "595-SN74AS04N" (at 242.57 203.2 0)
+      (effects (font (size 1.27 1.27)) hide)
+    )
+    (property "Alternative" "" (at 242.57 203.2 0)
       (effects (font (size 1.27 1.27)) hide)
     )
@@
       (effects (font (size 1.27 1.27)) hide)
     )
-    (property "Mouser" "" (at 93.726 70.612 0)
+    (property "Mouser" "595-SN74AS04N" (at 93.726 70.612 0)
+      (effects (font (size 1.27 1.27)) hide)
+    )
+    (property "Alternative" "" (at 93.726 70.612 0)
       (effects (font (size 1.27 1.27)) hide)
     )
