File: sheets/controller.kicad_sch (KiCad schematic)
At the start: 40 parts, among them CN1 CTRL1, CN2 CTRL2, U12 74LS06

Commit message: Schematics Footprint updates
Parts:
- CR1, CR2, CR3, CR4, CR5: footprint Resistor_THT:R_Array_SIP10 -> 1_NeoGeoLibrary:R_Array_SIP10
- U12: footprint Package_DIP:DIP-14_W7.62mm -> 1_NeoGeoLibrary:DIP-14_W7.62mm
Changed lines of the file:
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@@
       (effects (font (size 1.27 1.27)))
     )
-    (property "Footprint" "Package_DIP:DIP-14_W7.62mm" (at 243.586 128.27 0)
+    (property "Footprint" "1_NeoGeoLibrary:DIP-14_W7.62mm" (at 243.586 128.27 0)
       (effects (font (size 1.27 1.27)) hide)
     )
@@
       (effects (font (size 1.27 1.27)))
     )
-    (property "Footprint" "Resistor_THT:R_Array_SIP10" (at 109.474 189.23 0)
+    (property "Footprint" "1_NeoGeoLibrary:R_Array_SIP10" (at 109.474 189.23 0)
       (effects (font (size 1.27 1.27)) hide)
     )
@@
       (effects (font (size 1.27 1.27)))
     )
-    (property "Footprint" "Resistor_THT:R_Array_SIP10" (at 109.474 162.56 0)
+    (property "Footprint" "1_NeoGeoLibrary:R_Array_SIP10" (at 109.474 162.56 0)
       (effects (font (size 1.27 1.27)) hide)
     )
@@
       (effects (font (size 1.27 1.27)))
     )
-    (property "Footprint" "Package_DIP:DIP-14_W7.62mm" (at 243.586 184.404 0)
+    (property "Footprint" "1_NeoGeoLibrary:DIP-14_W7.62mm" (at 243.586 184.404 0)
       (effects (font (size 1.27 1.27)) hide)
     )
@@
       (effects (font (size 1.27 1.27)))
     )
-    (property "Footprint" "Resistor_THT:R_Array_SIP10" (at 109.474 215.9 0)
+    (property "Footprint" "1_NeoGeoLibrary:R_Array_SIP10" (at 109.474 215.9 0)
       (effects (font (size 1.27 1.27)) hide)
     )
@@
       (effects (font (size 1.27 1.27)))
     )
-    (property "Footprint" "Package_DIP:DIP-14_W7.62mm" (at 243.586 99.314 0)
+    (property "Footprint" "1_NeoGeoLibrary:DIP-14_W7.62mm" (at 243.586 99.314 0)
       (effects (font (size 1.27 1.27)) hide)
     )
@@
       (effects (font (size 1.27 1.27)))
     )
-    (property "Footprint" "Package_DIP:DIP-14_W7.62mm" (at 243.586 113.792 0)
+    (property "Footprint" "1_NeoGeoLibrary:DIP-14_W7.62mm" (at 243.586 113.792 0)
       (effects (font (size 1.27 1.27)) hide)
     )
@@
       (effects (font (size 1.27 1.27)))
     )
-    (property "Footprint" "Resistor_THT:R_Array_SIP10" (at 109.474 82.55 0)
+    (property "Footprint" "1_NeoGeoLibrary:R_Array_SIP10" (at 109.474 82.55 0)
       (effects (font (size 1.27 1.27)) hide)
     )
@@
       (effects (font (size 1.27 1.27)))
     )
-    (property "Footprint" "Package_DIP:DIP-14_W7.62mm" (at 243.586 213.36 0)
+    (property "Footprint" "1_NeoGeoLibrary:DIP-14_W7.62mm" (at 243.586 213.36 0)
       (effects (font (size 1.27 1.27)) hide)
     )
@@
       (effects (font (size 1.27 1.27)))
     )
-    (property "Footprint" "Resistor_THT:R_Array_SIP10" (at 109.474 109.22 0)
+    (property "Footprint" "1_NeoGeoLibrary:R_Array_SIP10" (at 109.474 109.22 0)
       (effects (font (size 1.27 1.27)) hide)
     )
@@
       (effects (font (size 1.27 1.27)))
     )
-    (property "Footprint" "Package_DIP:DIP-14_W7.62mm" (at 243.586 198.882 0)
-      (effects (font (size 1.27 1.27)) hide)
-    )
+    (property "Footprint" "1_NeoGeoLibrary:DIP-14_W7.62mm" (at 243.586 198.882 0)
+      (effects (font (size 1.27 1.27)) hide)
+    )

Commit message: Final update to Schematics Footprints Silkscreens
Parts:
- RN1: value 22Ω -> 22ΩX4
Changed lines of the file:
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@@
       (effects (font (size 1.27 1.27)))
     )
-    (property "Value" "22Ω" (at 262.89 124.968 90)
+    (property "Value" "22ΩX4" (at 262.89 124.968 90)
       (effects (font (size 1.27 1.27)))
     )
@@
       (effects (font (size 1.27 1.27)))
     )
-    (property "Value" "22Ω" (at 262.89 95.504 90)
+    (property "Value" "22ΩX4" (at 262.89 95.504 90)
       (effects (font (size 1.27 1.27)))
     )
@@
   (symbol (lib_id "Device:R_Pack04_SIP_Split") (at 262.89 113.792 90) (unit 2)
     (in_bom yes) (on_board yes) (dnp no) (fields_autoplaced)
-    (property "Reference" "RN1" (at 262.89 107.95 90)
-      (effects (font (size 1.27 1.27)))
-    )
-    (property "Value" "22Ω" (at 262.89 110.49 90)
-      (effects (font (size 1.27 1.27)))
-    )
+    (property "Reference" "RN1" (at 262.89 109.22 90)
+      (effects (font (size 1.27 1.27)))
+    )
+    (property "Value" "22ΩX4" (at 262.89 111.76 90)
+      (effects (font (size 1.27 1.27)))
+    )

Commit message: Some tweaks
Other:
- company: (none) -> SNK
- title: (none) -> NeoGeo AES
Changed lines of the file:
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@@
 (kicad_sch (version 20230121) (generator eeschema)
   (paper "A3")
+  (title_block
+    (title "NeoGeo AES")
+    (date "2023-08-19")
+    (rev "3.5")
+    (company "SNK")
+    (comment 3 "https://github.com/Board-Folk")
+    (comment 4 "Recreated By The Board Folk Team")
+  )
   (junction (at 131.572 139.7) (diameter 0) (color 0 0 0 0)
   )

Commit message: Updates to PCB Move P2 Joystick Port Move Memory Card Move Holes at top right Silkscreen added Update Titles
Other:
- title: NeoGeo AES -> NeoGeo AES 3-5
Changed lines of the file:
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@@
   (paper "A3")
   (title_block
-    (title "NeoGeo AES")
-    (date "2023-08-19")
-    (rev "3.5")
+    (title "NeoGeo AES 3-5")
+    (date "2023-08-27")
+    (rev "BF1.1")
     (company "SNK")
     (comment 3 "https://github.com/Board-Folk")

Commit message: Adding Mouser Part Numbers
Parts:
- BF1, BF10, BF11, BF12, BF13, BF14, BF15, BF16, BF17, BF18, BF19, BF2, BF20, BF21, BF22, BF23, BF24, BF25, BF26, BF27, BF28, BF29, BF3, BF30, BF4, BF5, BF6, BF7, BF8, BF9: Mouser (none) -> 80-B-06-R-25
Changed lines of the file:
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@@
+      (effects (font (size 1.27 1.27)) hide)
+    )
+    (property "Mouser" "80-B-06-R-25" (at 176.53 142.24 0)
       (effects (font (size 1.27 1.27)) hide)
     )
@@
     )
     (property "Datasheet" "" (at 243.586 128.27 0)
+      (effects (font (size 1.27 1.27)) hide)
+    )
+    (property "Mouser" "" (at 243.586 128.27 0)
       (effects (font (size 1.27 1.27)) hide)
     )
@@
       (effects (font (size 1.27 1.27)) hide)
     )
+    (property "Mouser" "" (at 109.474 189.23 0)
+      (effects (font (size 1.27 1.27)) hide)
+    )
     (pin "1")
     (pin "10")
@@
       (effects (font (size 1.27 1.27)) hide)
     )
+    (property "Mouser" "80-B-06-R-25" (at 176.53 151.13 0)
+      (effects (font (size 1.27 1.27)) hide)
+    )
     (pin "1")
     (pin "2")
@@
       (effects (font (size 1.27 1.27)) hide)
     )
+    (property "Mouser" "80-B-06-R-25" (at 157.734 88.9 0)
+      (effects (font (size 1.27 1.27)) hide)
+    )
     (pin "1")
     (pin "2")
@@
       (effects (font (size 1.27 1.27)) hide)
     )
+    (property "Mouser" "80-B-06-R-25" (at 176.53 168.91 0)
+      (effects (font (size 1.27 1.27)) hide)
+    )
     (pin "1")
     (pin "2")
@@
     )
     (property "Datasheet" "http://www.vishay.com/docs/31509/csc.pdf" (at 262.89 184.404 0)
+      (effects (font (size 1.27 1.27)) hide)
+    )
+    (property "Mouser" "" (at 262.89 184.404 0)
       (effects (font (size 1.27 1.27)) hide)
     )
@@
       (effects (font (size 1.27 1.27)) hide)
     )
+    (property "Mouser" "" (at 262.89 128.27 0)
+      (effects (font (size 1.27 1.27)) hide)
+    )
     (pin "1")
     (pin "2")
@@
       (effects (font (size 1.27 1.27)) hide)
     )
+    (property "Mouser" "80-B-06-R-25" (at 157.734 177.8 0)
+      (effects (font (size 1.27 1.27)) hide)
+    )
     (pin "1")
     (pin "2")
@@
       (effects (font (size 1.27 1.27)) hide)
     )
+    (property "Mouser" "80-B-06-R-25" (at 176.53 177.8 0)
+      (effects (font (size 1.27 1.27)) hide)
+    )
     (pin "1")
     (pin "2")
@@
       (effects (font (size 1.27 1.27)) hide)
     )
+    (property "Mouser" "80-B-06-R-25" (at 313.69 42.672 0)
+      (effects (font (size 1.27 1.27)) hide)
+    )
     (pin "1")
     (pin "2")
@@
       (effects (font (size 1.27 1.27)) hide)
     )
+    (property "Mouser" "80-B-06-R-25" (at 176.53 88.9 0)
+      (effects (font (size 1.27 1.27)) hide)
+    )
     (pin "1")
     (pin "2")
@@
       (effects (font (size 1.27 1.27)) hide)
     )
+    (property "Mouser" "" (at 109.474 162.56 0)
+      (effects (font (size 1.27 1.27)) hide)
+    )
     (pin "1")
     (pin "10")
@@
       (effects (font (size 1.27 1.27)) hide)
     )
+    (property "Mouser" "80-B-06-R-25" (at 157.734 151.13 0)
+      (effects (font (size 1.27 1.27)) hide)
+    )
     (pin "1")
     (pin "2")
@@
       (effects (font (size 1.27 1.27)) hide)
     )
+    (property "Mouser" "80-B-06-R-25" (at 176.53 97.79 0)
+      (effects (font (size 1.27 1.27)) hide)
+    )
     (pin "1")
     (pin "2")
@@
       (effects (font (size 1.27 1.27)) hide)
     )
+    (property "Mouser" "80-B-06-R-25" (at 313.69 112.268 0)
+      (effects (font (size 1.27 1.27)) hide)
+    )
     (pin "1")
     (pin "2")
@@
       (effects (font (size 1.27 1.27)) hide)
     )
+    (property "Mouser" "80-B-06-R-25" (at 271.526 128.27 0)
+      (effects (font (size 1.27 1.27)) hide)
+    )
     (pin "1")
     (pin "2")
@@
       (effects (font (size 1.27 1.27)) hide)
     )
+    (property "Mouser" "80-B-06-R-25" (at 176.53 204.47 0)
+      (effects (font (size 1.27 1.27)) hide)
+    )
     (pin "1")
     (pin "2")
@@
     )
     (property "Datasheet" "" (at 243.586 184.404 0)
+      (effects (font (size 1.27 1.27)) hide)
+    )
+    (property "Mouser" "" (at 243.586 184.404 0)
       (effects (font (size 1.27 1.27)) hide)
     )
@@
       (effects (font (size 1.27 1.27)) hide)
     )
+    (property "Mouser" "80-B-06-R-25" (at 157.734 204.47 0)
+      (effects (font (size 1.27 1.27)) hide)
+    )
     (pin "1")
     (pin "2")
@@
     )
     (property "Datasheet" "" (at 318.77 77.47 0)
+      (effects (font (size 1.27 1.27)) hide)
+    )
+    (property "Mouser" "" (at 318.77 77.47 0)
       (effects (font (size 1.27 1.27)) hide)
     )
@@
       (effects (font (size 1.27 1.27)) hide)
     )
+    (property "Mouser" "80-B-06-R-25" (at 157.734 97.79 0)
+      (effects (font (size 1.27 1.27)) hide)
+    )
     (pin "1")
     (pin "2")
@@
     )
     (property "Datasheet" "" (at 109.474 215.9 0)
+      (effects (font (size 1.27 1.27)) hide)
+    )
+    (property "Mouser" "" (at 109.474 215.9 0)
       (effects (font (size 1.27 1.27)) hide)
     )
@@
       (effects (font (size 1.27 1.27)) hide)
     )
+    (property "Mouser" "" (at 262.89 213.36 0)
+      (effects (font (size 1.27 1.27)) hide)
+    )
     (pin "1")
     (pin "2")
@@
       (effects (font (size 1.27 1.27)) hide)
     )
+    (property "Mouser" "" (at 262.89 99.314 0)
+      (effects (font (size 1.27 1.27)) hide)
+    )
     (pin "1")
     (pin "2")
@@
     )
     (property "Datasheet" "" (at 318.77 162.56 0)
+      (effects (font (size 1.27 1.27)) hide)
+    )
+    (property "Mouser" "" (at 318.77 162.56 0)
       (effects (font (size 1.27 1.27)) hide)
     )
@@
       (effects (font (size 1.27 1.27)) hide)
     )
+    (property "Mouser" "80-B-06-R-25" (at 157.734 62.23 0)
+      (effects (font (size 1.27 1.27)) hide)
+    )
     (pin "1")
     (pin "2")
@@
       (effects (font (size 1.27 1.27)) hide)
     )
+    (property "Mouser" "80-B-06-R-25" (at 176.53 71.12 0)
+      (effects (font (size 1.27 1.27)) hide)
+    )
     (pin "1")
     (pin "2")
@@
       (effects (font (size 1.27 1.27)) hide)
     )
+    (property "Mouser" "80-B-06-R-25" (at 271.526 213.36 0)
+      (effects (font (size 1.27 1.27)) hide)
+    )
     (pin "1")
     (pin "2")
@@
       (effects (font (size 1.27 1.27)) hide)
     )
+    (property "Mouser" "80-B-06-R-25" (at 313.69 197.358 0)
+      (effects (font (size 1.27 1.27)) hide)
+    )
     (pin "1")
     (pin "2")
@@
     )
     (property "Datasheet" "" (at 271.526 198.882 0)
+      (effects (font (size 1.27 1.27)) hide)
+    )
+    (property "Mouser" "80-B-06-R-25" (at 271.526 198.882 0)
       (effects (font (size 1.27 1.27)) hide)
     )
@@
       (effects (font (size 1.27 1.27)) hide)
     )
+    (property "Mouser" "" (at 262.89 113.792 0)
+      (effects (font (size 1.27 1.27)) hide)
+    )
     (pin "1")
     (pin "2")
@@
       (effects (font (size 1.27 1.27)) hide)
     )
+    (property "Mouser" "80-B-06-R-25" (at 176.53 195.58 0)
+      (effects (font (size 1.27 1.27)) hide)
+    )
     (pin "1")
     (pin "2")
@@
       (effects (font (size 1.27 1.27)) hide)
     )
+    (property "Mouser" "80-B-06-R-25" (at 157.734 142.24 0)
+      (effects (font (size 1.27 1.27)) hide)
+    )
     (pin "1")
     (pin "2")
@@
       (effects (font (size 1.27 1.27)) hide)
     )
+    (property "Mouser" "80-B-06-R-25" (at 157.734 195.58 0)
+      (effects (font (size 1.27 1.27)) hide)
+    )
     (pin "1")
     (pin "2")
@@
     )
     (property "Datasheet" "" (at 243.586 99.314 0)
+      (effects (font (size 1.27 1.27)) hide)
+    )
+    (property "Mouser" "" (at 243.586 99.314 0)
       (effects (font (size 1.27 1.27)) hide)
     )
@@
       (effects (font (size 1.27 1.27)) hide)
     )
+    (property "Mouser" "80-B-06-R-25" (at 157.734 71.12 0)
+      (effects (font (size 1.27 1.27)) hide)
+    )
     (pin "1")
     (pin "2")
@@
     )
     (property "Datasheet" "" (at 243.586 113.792 0)
+      (effects (font (size 1.27 1.27)) hide)
+    )
+    (property "Mouser" "" (at 243.586 113.792 0)
       (effects (font (size 1.27 1.27)) hide)
     )
@@
       (effects (font (size 1.27 1.27)) hide)
     )
+    (property "Mouser" "80-B-06-R-25" (at 313.69 127.762 0)
+      (effects (font (size 1.27 1.27)) hide)
+    )
     (pin "1")
     (pin "2")
@@
     )
     (property "Datasheet" "" (at 271.526 184.404 0)
+      (effects (font (size 1.27 1.27)) hide)
+    )
+    (property "Mouser" "80-B-06-R-25" (at 271.526 184.404 0)
       (effects (font (size 1.27 1.27)) hide)
     )
@@
       (effects (font (size 1.27 1.27)) hide)
     )
+    (property "Mouser" "" (at 262.89 198.882 0)
+      (effects (font (size 1.27 1.27)) hide)
+    )
     (pin "1")
     (pin "2")
@@
       (effects (font (size 1.27 1.27)) hide)
     )
+    (property "Mouser" "80-B-06-R-25" (at 157.734 168.91 0)
+      (effects (font (size 1.27 1.27)) hide)
+    )
     (pin "1")
     (pin "2")
@@
       (effects (font (size 1.27 1.27)) hide)
     )
+    (property "Mouser" "" (at 109.474 82.55 0)
+      (effects (font (size 1.27 1.27)) hide)
+    )
     (pin "1")
     (pin "10")
@@
       (effects (font (size 1.27 1.27)) hide)
     )
+    (property "Mouser" "80-B-06-R-25" (at 271.526 113.792 0)
+      (effects (font (size 1.27 1.27)) hide)
+    )
     (pin "1")
     (pin "2")
@@
     )
     (property "Datasheet" "" (at 243.586 213.36 0)
+      (effects (font (size 1.27 1.27)) hide)
+    )
+    (property "Mouser" "" (at 243.586 213.36 0)
       (effects (font (size 1.27 1.27)) hide)
     )
@@
       (effects (font (size 1.27 1.27)) hide)
     )
+    (property "Mouser" "" (at 109.474 109.22 0)
+      (effects (font (size 1.27 1.27)) hide)
+    )
     (pin "1")
     (pin "10")
@@
     )
     (property "Datasheet" "" (at 243.586 198.882 0)
+      (effects (font (size 1.27 1.27)) hide)
+    )
+    (property "Mouser" "" (at 243.586 198.882 0)
       (effects (font (size 1.27 1.27)) hide)
     )
@@
       (effects (font (size 1.27 1.27)) hide)
     )
+    (property "Mouser" "80-B-06-R-25" (at 271.526 99.314 0)
+      (effects (font (size 1.27 1.27)) hide)
+    )
     (pin "1")
     (pin "2")
@@
       (effects (font (size 1.27 1.27)) hide)
     )
+    (property "Mouser" "80-B-06-R-25" (at 176.53 62.23 0)
+      (effects (font (size 1.27 1.27)) hide)
+    )

Commit message: More silkscreen tidy up, adding mouser components to BOM
Parts:
- CR1, CR2, CR3, CR4, CR5: Comment (none) -> https://github.com/mourix/CRE401
- RN1: value 22ΩX4 -> 22x4
- RN2: value 22Ω -> 22
Changed lines of the file:
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@@
+      (effects (font (size 1.27 1.27)) hide)
+    )
+    (property "Comment" "https://github.com/mourix/CRE401" (at 109.474 189.23 0)
       (effects (font (size 1.27 1.27)) hide)
     )
@@
       (effects (font (size 1.27 1.27)))
     )
-    (property "Value" "22Ω" (at 262.89 181.102 90)
+    (property "Value" "22" (at 262.89 181.102 90)
       (effects (font (size 1.27 1.27)))
     )
@@
       (effects (font (size 1.27 1.27)))
     )
-    (property "Value" "22ΩX4" (at 262.89 124.968 90)
+    (property "Value" "22x4" (at 262.89 124.968 90)
       (effects (font (size 1.27 1.27)))
     )
@@
     )
     (property "Mouser" "" (at 109.474 162.56 0)
+      (effects (font (size 1.27 1.27)) hide)
+    )
+    (property "Comment" "https://github.com/mourix/CRE401" (at 109.474 162.56 0)
       (effects (font (size 1.27 1.27)) hide)
     )
@@
       (effects (font (size 1.27 1.27)) hide)
     )
+    (property "Comment" "https://github.com/mourix/CRE401" (at 109.474 215.9 0)
+      (effects (font (size 1.27 1.27)) hide)
+    )
     (pin "1")
     (pin "10")
@@
       (effects (font (size 1.27 1.27)))
     )
-    (property "Value" "22Ω" (at 262.89 209.296 90)
+    (property "Value" "22" (at 262.89 209.296 90)
       (effects (font (size 1.27 1.27)))
     )
@@
       (effects (font (size 1.27 1.27)))
     )
-    (property "Value" "22ΩX4" (at 262.89 95.504 90)
+    (property "Value" "22x4" (at 262.89 95.504 90)
       (effects (font (size 1.27 1.27)))
     )
@@
       (effects (font (size 1.27 1.27)))
     )
-    (property "Value" "22ΩX4" (at 262.89 111.76 90)
+    (property "Value" "22x4" (at 262.89 111.76 90)
       (effects (font (size 1.27 1.27)))
     )
@@
       (effects (font (size 1.27 1.27)))
     )
-    (property "Value" "22Ω" (at 262.89 194.564 90)
+    (property "Value" "22" (at 262.89 194.564 90)
       (effects (font (size 1.27 1.27)))
     )
@@
     )
     (property "Mouser" "" (at 109.474 82.55 0)
+      (effects (font (size 1.27 1.27)) hide)
+    )
+    (property "Comment" "https://github.com/mourix/CRE401" (at 109.474 82.55 0)
       (effects (font (size 1.27 1.27)) hide)
     )
@@
       (effects (font (size 1.27 1.27)) hide)
     )
+    (property "Comment" "https://github.com/mourix/CRE401" (at 109.474 109.22 0)
+      (effects (font (size 1.27 1.27)) hide)
+    )

Commit message: Little tweaks to silkscreen Updated BOM with mouser parts
Parts:
- CN1, CN2: Comment (none) -> Use Original
- CR1, CR2, CR3, CR4, CR5: Alternative (none) -> https://github.com/mourix/CRE401; Comment https://github.com/mourix/CRE401 -> (none)
- RN1: Mouser (none) -> 652-4608X-2LF-22
- RN2: value 22 -> 22x4; Mouser (none) -> 652-4608X-2LF-22
- U12: Mouser (none) -> 595-SN74LS06N
