File: sheets/ym2610_audio.kicad_sch (KiCad schematic)
At the start: 56 parts, among them J3 SMK S-G8043, Q101 2SC1815, Q102 2SC1815, U26 YM3016D, U27 YM2610, U28 PC4741, U29 PC4741

Commit message: update before public
Parts:
- R301, R32, R36, R37, R38, R39, R40, R41, R42, R43, R45: Mouser 71-CMF501K0000FHEA -> (none)
- R302: Mouser 71-RN60D-F-30K -> (none)
- R303: Mouser 71-RN60E1002F -> (none)
- R31: Mouser 71-RN60D4701F -> (none)
- R33, R34: Mouser 71-CMF5010R000FHEK -> (none)
- R401, R501: Mouser 71-CMF5075R000FHEB -> (none)
- R402, R502: Mouser 71-RN60D5102F -> (none)
- R403, R503: Mouser 71-CMF5015K000FHEK -> (none)
- R46, R49: Mouser 71-RN60D-F-27K -> (none)
- R47, R48: Mouser 71-RN60D4702F -> (none)
Changed lines of the file:
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@@
       (effects (font (size 1.27 1.27)) hide)
     )
-    (property "Mouser" "71-CMF501K0000FHEA" (at 166.751 208.153 0)
+    (property "Mouser" "" (at 166.751 208.153 0)
       (effects (font (size 1.27 1.27)) hide)
     )
@@
       (effects (font (size 1.27 1.27)) hide)
     )
-    (property "Mouser" "71-RN60E1002F" (at 334.264 95.25 0)
+    (property "Mouser" "" (at 334.264 95.25 0)
       (effects (font (size 1.27 1.27)) hide)
     )
@@
       (effects (font (size 1.27 1.27)) hide)
     )
-    (property "Mouser" "71-CMF501K0000FHEA" (at 166.751 227.203 0)
+    (property "Mouser" "" (at 166.751 227.203 0)
       (effects (font (size 1.27 1.27)) hide)
     )
@@
       (effects (font (size 1.27 1.27)) hide)
     )
-    (property "Mouser" "71-RN60D5102F" (at 222.885 206.883 0)
+    (property "Mouser" "" (at 222.885 206.883 0)
       (effects (font (size 1.27 1.27)) hide)
     )
@@
       (effects (font (size 1.27 1.27)) hide)
     )
-    (property "Mouser" "71-CMF501K0000FHEA" (at 307.086 81.661 0)
+    (property "Mouser" "" (at 307.086 81.661 0)
       (effects (font (size 1.27 1.27)) hide)
     )
@@
       (effects (font (size 1.27 1.27)) hide)
     )
-    (property "Mouser" "71-CMF5015K000FHEK" (at 222.885 230.378 0)
+    (property "Mouser" "" (at 222.885 230.378 0)
       (effects (font (size 1.27 1.27)) hide)
     )
@@
       (effects (font (size 1.27 1.27)) hide)
     )
-    (property "Mouser" "71-CMF501K0000FHEA" (at 307.086 83.693 0)
+    (property "Mouser" "" (at 307.086 83.693 0)
       (effects (font (size 1.27 1.27)) hide)
     )
@@
       (effects (font (size 1.27 1.27)) hide)
     )
-    (property "Mouser" "71-RN60D4702F" (at 117.221 210.693 0)
+    (property "Mouser" "" (at 117.221 210.693 0)
       (effects (font (size 1.27 1.27)) hide)
     )
@@
       (effects (font (size 1.27 1.27)) hide)
     )
-    (property "Mouser" "71-CMF501K0000FHEA" (at 271.018 58.801 0)
+    (property "Mouser" "" (at 271.018 58.801 0)
       (effects (font (size 1.27 1.27)) hide)
     )
@@
       (effects (font (size 1.27 1.27)) hide)
     )
-    (property "Mouser" "71-RN60D-F-27K" (at 117.221 198.374 0)
+    (property "Mouser" "" (at 117.221 198.374 0)
       (effects (font (size 1.27 1.27)) hide)
     )
@@
       (effects (font (size 1.27 1.27)) hide)
     )
-    (property "Mouser" "71-CMF5010R000FHEK" (at 239.776 226.568 0)
+    (property "Mouser" "" (at 239.776 226.568 0)
       (effects (font (size 1.27 1.27)) hide)
     )
@@
       (effects (font (size 1.27 1.27)) hide)
     )
-    (property "Mouser" "71-CMF5010R000FHEK" (at 239.776 208.788 0)
+    (property "Mouser" "" (at 239.776 208.788 0)
       (effects (font (size 1.27 1.27)) hide)
     )
@@
       (effects (font (size 1.27 1.27)) hide)
     )
-    (property "Mouser" "71-CMF5075R000FHEB" (at 222.885 226.568 0)
+    (property "Mouser" "" (at 222.885 226.568 0)
       (effects (font (size 1.27 1.27)) hide)
     )
@@
       (effects (font (size 1.27 1.27)) hide)
     )
-    (property "Mouser" "71-CMF501K0000FHEA" (at 271.018 81.661 0)
+    (property "Mouser" "" (at 271.018 81.661 0)
       (effects (font (size 1.27 1.27)) hide)
     )
@@
       (effects (font (size 1.27 1.27)) hide)
     )
-    (property "Mouser" "71-RN60D4701F" (at 69.596 90.551 0)
+    (property "Mouser" "" (at 69.596 90.551 0)
       (effects (font (size 1.27 1.27)) hide)
     )
@@
       (effects (font (size 1.27 1.27)) hide)
     )
-    (property "Mouser" "71-CMF501K0000FHEA" (at 287.782 81.661 0)
+    (property "Mouser" "" (at 287.782 81.661 0)
       (effects (font (size 1.27 1.27)) hide)
     )
@@
       (effects (font (size 1.27 1.27)) hide)
     )
-    (property "Mouser" "71-CMF501K0000FHEA" (at 287.782 58.801 0)
+    (property "Mouser" "" (at 287.782 58.801 0)
       (effects (font (size 1.27 1.27)) hide)
     )
@@
       (effects (font (size 1.27 1.27)) hide)
     )
-    (property "Mouser" "71-RN60D4702F" (at 117.221 224.663 0)
+    (property "Mouser" "" (at 117.221 224.663 0)
       (effects (font (size 1.27 1.27)) hide)
     )
@@
       (effects (font (size 1.27 1.27)) hide)
     )
-    (property "Mouser" "71-CMF5015K000FHEK" (at 222.885 204.978 0)
+    (property "Mouser" "" (at 222.885 204.978 0)
       (effects (font (size 1.27 1.27)) hide)
     )
@@
       (effects (font (size 1.27 1.27)) hide)
     )
-    (property "Mouser" "71-RN60D5102F" (at 222.885 228.473 0)
+    (property "Mouser" "" (at 222.885 228.473 0)
       (effects (font (size 1.27 1.27)) hide)
     )
@@
       (effects (font (size 1.27 1.27)) hide)
     )
-    (property "Mouser" "71-CMF501K0000FHEA" (at 307.086 85.725 0)
+    (property "Mouser" "" (at 307.086 85.725 0)
       (effects (font (size 1.27 1.27)) hide)
     )
@@
       (effects (font (size 1.27 1.27)) hide)
     )
-    (property "Mouser" "71-CMF501K0000FHEA" (at 128.905 147.066 0)
+    (property "Mouser" "" (at 128.905 147.066 0)
       (effects (font (size 1.27 1.27)) hide)
     )
@@
       (effects (font (size 1.27 1.27)) hide)
     )
-    (property "Mouser" "71-CMF501K0000FHEA" (at 226.822 53.721 0)
+    (property "Mouser" "" (at 226.822 53.721 0)
       (effects (font (size 1.27 1.27)) hide)
     )
@@
       (effects (font (size 1.27 1.27)) hide)
     )
-    (property "Mouser" "71-RN60D-F-30K" (at 334.264 88.265 0)
+    (property "Mouser" "" (at 334.264 88.265 0)
       (effects (font (size 1.27 1.27)) hide)
     )
@@
       (effects (font (size 1.27 1.27)) hide)
     )
-    (property "Mouser" "71-CMF5075R000FHEB" (at 222.885 208.788 0)
+    (property "Mouser" "" (at 222.885 208.788 0)
       (effects (font (size 1.27 1.27)) hide)
     )
@@
       (effects (font (size 1.27 1.27)) hide)
     )
-    (property "Mouser" "71-RN60D-F-27K" (at 117.221 236.982 0)
-      (effects (font (size 1.27 1.27)) hide)
-    )
+    (property "Mouser" "" (at 117.221 236.982 0)
+      (effects (font (size 1.27 1.27)) hide)
+    )
