File: sheets/cpu.kicad_sch (KiCad schematic)
At the start: 6 parts, among them J1 BERR, U1 uPD43256AGU-12L, U2 uPD43256AGU-12L, U3 HD68HC000P, U4 NEO-C1

Commit message: Update BF1.4
Update Mouser Parts
Update Silkscreen for Memory Slot
Update Silkscreen for BF1.4 Version and date
Generate Gerbers and BOM files
Parts:
- U1, U2: Alternative (none) -> JEDEC 62256 (32k x 8) SRAM; Mouser (none) -> 870-62C256AL-25ULI
Changed lines of the file:
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@@
   (title_block
     (title "NeoGeo AES 3-5")
-    (date "2023-12-30")
-    (rev "BF1.3")
+    (date "2024-01-06")
+    (rev "BF1.4")
     (company "SNK")
     (comment 3 "https://github.com/Board-Folk")
@@
       (effects (font (size 1.27 1.27)) hide)
     )
-    (property "Mouser" "" (at 197.612 118.618 0)
-      (effects (font (size 1.27 1.27)) hide)
-    )
-    (property "Alternative" "" (at 197.612 118.618 0)
+    (property "Mouser" "870-62C256AL-25ULI" (at 197.612 118.618 0)
+      (effects (font (size 1.27 1.27)) hide)
+    )
+    (property "Alternative" "JEDEC 62256 (32k x 8) SRAM" (at 197.612 118.618 0)
       (effects (font (size 1.27 1.27)) hide)
     )
@@
       (effects (font (size 1.27 1.27)) hide)
     )
-    (property "Mouser" "" (at 197.612 169.672 0)
-      (effects (font (size 1.27 1.27)) hide)
-    )
-    (property "Alternative" "" (at 197.612 169.672 0)
-      (effects (font (size 1.27 1.27)) hide)
-    )
+    (property "Mouser" "870-62C256AL-25ULI" (at 197.612 169.672 0)
+      (effects (font (size 1.27 1.27)) hide)
+    )
+    (property "Alternative" "JEDEC 62256 (32k x 8) SRAM" (at 197.612 169.672 0)
+      (effects (font (size 1.27 1.27)) hide)
+    )

Commit message: Update Silk
Update Ram Silk
Fix mouser wrong 6.8K
Update BOM, Gerbers ...
Parts:
- U1, U2: value uPD43256AGU-12L -> 43256
Changed lines of the file:
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@@
       (effects (font (size 1.27 1.27)) (justify left))
     )
-    (property "Value" "uPD43256AGU-12L" (at 197.5612 122.174 90)
+    (property "Value" "43256" (at 197.612 117.348 90)
       (effects (font (size 1.27 1.27)) (justify left))
     )
@@
       (effects (font (size 1.27 1.27)) (justify left))
     )
-    (property "Value" "uPD43256AGU-12L" (at 197.5612 173.228 90)
-      (effects (font (size 1.27 1.27)) (justify left))
-    )
+    (property "Value" "43256" (at 197.612 168.402 90)
+      (effects (font (size 1.27 1.27)) (justify left))
+    )
