File: sheets/rgb_video.kicad_sch (KiCad schematic)
At the start: 51 parts, among them CN3 DIN-8, U32 CXA1145P

Commit message: Update BF1.4
Update Mouser Parts
Update Silkscreen for Memory Slot
Update Silkscreen for BF1.4 Version and date
Generate Gerbers and BOM files
Parts:
- C36, C37, C38, C39: Mouser 647-UHE1C471MPD6 -> 647-UVR1C471MPD1TA
- C43: Mouser 810-FG28C0G1H101JNT6 -> 810-FG28C0G1H470JNT6
- R50, R51, R52, R75: Mouser (none) -> 594-5063JD3K000F
- R53: Mouser (none) -> 594-5063JD27K00FT
- R54, R55: Mouser 71-CMF501K0000FHEA -> 594-5063JD1K000FT
- R56: Mouser (none) -> 594-5063JD820R0FT
- R57: Mouser (none) -> 594-5063JD10K1%TR
- R58, R59, R60: Mouser (none) -> 594-5063JD75R00F
- R62, R63, R64, R65: Mouser 71-CMF5075R000FHEB -> 594-5063JD75R00FT
- R66: Mouser (none) -> 594-5063JD470R0FT
- U32: Alternative (none) -> CXA1645 or CXA2075 needs adapter
Changed lines of the file:
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@@
   (title_block
     (title "NeoGeo AES 3-5")
-    (date "2023-12-30")
-    (rev "BF1.3")
+    (date "2024-01-06")
+    (rev "BF1.4")
     (company "SNK")
     (comment 3 "https://github.com/Board-Folk")
@@
       (effects (font (size 1.27 1.27)) hide)
     )
-    (property "Mouser" "71-CMF5075R000FHEB" (at 268.478 112.776 0)
+    (property "Mouser" "594-5063JD75R00FT" (at 268.478 112.776 0)
       (effects (font (size 1.27 1.27)) hide)
     )
@@
       (effects (font (size 1.27 1.27)) hide)
     )
-    (property "Mouser" "" (at 95.25 127.254 0)
+    (property "Mouser" "594-5063JD3K000F" (at 95.25 127.254 0)
       (effects (font (size 1.27 1.27)) hide)
     )
@@
       (effects (font (size 1.27 1.27)) hide)
     )
-    (property "Mouser" "" (at 95.25 104.394 0)
+    (property "Mouser" "594-5063JD3K000F" (at 95.25 104.394 0)
       (effects (font (size 1.27 1.27)) hide)
     )
@@
       (effects (font (size 1.27 1.27)) hide)
     )
-    (property "Alternative" "" (at 213.106 179.578 0)
+    (property "Alternative" "CXA1645 or CXA2075 needs adapter" (at 213.106 179.578 0)
       (effects (font (size 1.27 1.27)) hide)
     )
@@
       (effects (font (size 1.27 1.27)) hide)
     )
-    (property "Mouser" "71-CMF5075R000FHEB" (at 268.478 100.584 0)
+    (property "Mouser" "594-5063JD75R00FT" (at 268.478 100.584 0)
       (effects (font (size 1.27 1.27)) hide)
     )
@@
       (effects (font (size 1.27 1.27)) hide)
     )
-    (property "Mouser" "" (at 89.408 121.412 0)
+    (property "Mouser" "594-5063JD75R00F" (at 89.408 121.412 0)
       (effects (font (size 1.27 1.27)) hide)
     )
@@
       (effects (font (size 1.27 1.27)) hide)
     )
-    (property "Mouser" "71-CMF5075R000FHEB" (at 268.478 88.392 0)
+    (property "Mouser" "594-5063JD75R00FT" (at 268.478 88.392 0)
       (effects (font (size 1.27 1.27)) hide)
     )
@@
       (effects (font (size 1.27 1.27)) hide)
     )
-    (property "Mouser" "" (at 89.408 98.552 0)
+    (property "Mouser" "594-5063JD75R00F" (at 89.408 98.552 0)
       (effects (font (size 1.27 1.27)) hide)
     )
@@
       (effects (font (size 1.27 1.27)) hide)
     )
-    (property "Mouser" "71-CMF501K0000FHEA" (at 248.412 183.896 0)
+    (property "Mouser" "594-5063JD1K000FT" (at 248.412 183.896 0)
       (effects (font (size 1.27 1.27)) hide)
     )
@@
       (effects (font (size 1.27 1.27)) hide)
     )
-    (property "Mouser" "" (at 259.334 205.232 0)
+    (property "Mouser" "594-5063JD820R0FT" (at 259.334 205.232 0)
       (effects (font (size 1.27 1.27)) hide)
     )
@@
       (effects (font (size 1.27 1.27)) hide)
     )
-    (property "Mouser" "71-CMF501K0000FHEA" (at 266.446 154.686 0)
+    (property "Mouser" "594-5063JD1K000FT" (at 266.446 154.686 0)
       (effects (font (size 1.27 1.27)) hide)
     )
@@
       (effects (font (size 1.27 1.27)) hide)
     )
-    (property "Mouser" "" (at 181.61 180.848 0)
+    (property "Mouser" "594-5063JD27K00FT" (at 181.61 180.848 0)
       (effects (font (size 1.27 1.27)) hide)
     )
@@
       (effects (font (size 1.27 1.27)) hide)
     )
-    (property "Mouser" "" (at 282.194 168.656 0)
+    (property "Mouser" "594-5063JD470R0FT" (at 282.194 168.656 0)
       (effects (font (size 1.27 1.27)) hide)
     )
@@
       (effects (font (size 1.27 1.27)) hide)
     )
-    (property "Mouser" "" (at 95.25 150.114 0)
+    (property "Mouser" "594-5063JD3K000F" (at 95.25 150.114 0)
       (effects (font (size 1.27 1.27)) hide)
     )
@@
       (effects (font (size 1.27 1.27)) hide)
     )
-    (property "Mouser" "810-FG28C0G1H101JNT6" (at 292.1 168.656 0)
+    (property "Mouser" "810-FG28C0G1H470JNT6" (at 292.1 168.656 0)
       (effects (font (size 1.27 1.27)) hide)
     )
@@
       (effects (font (size 1.27 1.27)) hide)
     )
-    (property "Mouser" "" (at 89.408 144.272 0)
+    (property "Mouser" "594-5063JD75R00F" (at 89.408 144.272 0)
       (effects (font (size 1.27 1.27)) hide)
     )
@@
       (effects (font (size 1.27 1.27)) hide)
     )
-    (property "Mouser" "647-UHE1C471MPD6" (at 253.492 112.776 0)
+    (property "Mouser" "647-UVR1C471MPD1TA" (at 253.492 112.776 0)
       (effects (font (size 1.27 1.27)) hide)
     )
@@
       (effects (font (size 1.27 1.27)) hide)
     )
-    (property "Mouser" "647-UHE1C471MPD6" (at 253.492 76.708 0)
+    (property "Mouser" "647-UVR1C471MPD1TA" (at 253.492 76.708 0)
       (effects (font (size 1.27 1.27)) hide)
     )
@@
       (effects (font (size 1.27 1.27)) hide)
     )
-    (property "Mouser" "" (at 125.222 170.688 0)
+    (property "Mouser" "594-5063JD3K000F" (at 125.222 170.688 0)
       (effects (font (size 1.27 1.27)) hide)
     )
@@
       (effects (font (size 1.27 1.27)) hide)
     )
-    (property "Mouser" "647-UHE1C471MPD6" (at 253.492 100.584 0)
+    (property "Mouser" "647-UVR1C471MPD1TA" (at 253.492 100.584 0)
       (effects (font (size 1.27 1.27)) hide)
     )
@@
       (effects (font (size 1.27 1.27)) hide)
     )
-    (property "Mouser" "647-UHE1C471MPD6" (at 253.492 88.392 0)
+    (property "Mouser" "647-UVR1C471MPD1TA" (at 253.492 88.392 0)
       (effects (font (size 1.27 1.27)) hide)
     )
@@
       (effects (font (size 1.27 1.27)) hide)
     )
-    (property "Mouser" "" (at 261.493 122.682 0)
+    (property "Mouser" "594-5063JD10K1%TR" (at 261.493 122.682 0)
       (effects (font (size 1.27 1.27)) hide)
     )
@@
       (effects (font (size 1.27 1.27)) hide)
     )
-    (property "Mouser" "71-CMF5075R000FHEB" (at 268.478 76.708 0)
-      (effects (font (size 1.27 1.27)) hide)
-    )
+    (property "Mouser" "594-5063JD75R00FT" (at 268.478 76.708 0)
+      (effects (font (size 1.27 1.27)) hide)
+    )

Commit message: Update Silk
Update Ram Silk
Fix mouser wrong 6.8K
Update BOM, Gerbers ...
Parts:
- R58, R59, R60: Mouser 594-5063JD75R00F -> 594-5063JD6R800F5
Changed lines of the file:
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@@
       (effects (font (size 1.27 1.27)) hide)
     )
-    (property "Mouser" "594-5063JD75R00F" (at 89.408 121.412 0)
+    (property "Mouser" "594-5063JD6R800F5" (at 89.408 121.412 0)
       (effects (font (size 1.27 1.27)) hide)
     )
@@
       (effects (font (size 1.27 1.27)) hide)
     )
-    (property "Mouser" "594-5063JD75R00F" (at 89.408 98.552 0)
+    (property "Mouser" "594-5063JD6R800F5" (at 89.408 98.552 0)
       (effects (font (size 1.27 1.27)) hide)
     )
@@
       (effects (font (size 1.27 1.27)) hide)
     )
-    (property "Mouser" "594-5063JD75R00F" (at 89.408 144.272 0)
-      (effects (font (size 1.27 1.27)) hide)
-    )
+    (property "Mouser" "594-5063JD6R800F5" (at 89.408 144.272 0)
+      (effects (font (size 1.27 1.27)) hide)
+    )

Commit message: fix wrong mouser part for 6.8K Resistor
Parts:
- R58, R59, R60: Mouser 594-5063JD6R800F5 -> 594-5063JD6K810FT
Changed lines of the file:
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@@
       (effects (font (size 1.27 1.27)) hide)
     )
-    (property "Mouser" "594-5063JD6R800F5" (at 89.408 121.412 0)
+    (property "Mouser" "594-5063JD6K810FT" (at 89.408 121.412 0)
       (effects (font (size 1.27 1.27)) hide)
     )
@@
       (effects (font (size 1.27 1.27)) hide)
     )
-    (property "Mouser" "594-5063JD6R800F5" (at 89.408 98.552 0)
+    (property "Mouser" "594-5063JD6K810FT" (at 89.408 98.552 0)
       (effects (font (size 1.27 1.27)) hide)
     )
@@
       (effects (font (size 1.27 1.27)) hide)
     )
-    (property "Mouser" "594-5063JD6R800F5" (at 89.408 144.272 0)
-      (effects (font (size 1.27 1.27)) hide)
-    )
+    (property "Mouser" "594-5063JD6K810FT" (at 89.408 144.272 0)
+      (effects (font (size 1.27 1.27)) hide)
+    )
