File: sheets/graphics.kicad_sch (KiCad schematic)
At the start: 25 parts, among them J2 CUT DOG, SW1 RESET SWITCH, U13 NEO-B1, U14 PST518B, U15 74LS244, U16 TC531000AP, U17 43256, U18 43256, U19 5863 / 5814, U20 5863 / 5814, U21 LSPC2

Commit message: Updated to Kicad 10
Connections:
- net GND: now also U21.83 (GND); no longer U21.93 (GND)
Other:
- moved on the sheet: C1, C56, C57, C58, C59, C61, C62, PAL1, R28, R29, R5814, R5863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
