File: NeoGeoAES3_5.kicad_sch (KiCad schematic)
At the start: 0 parts

Commit message: Renamed SDD[0..15] to SDD[0..7]
Other:
- sheet Cartridge Slots ports: added SDD[0..7]; removed SDD[0..15]
Changed lines of the file:
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@@
       (effects (font (size 1.27 1.27)) (justify right))
     )
-    (pin "SDD[0..15]" input (at 322.58 91.44 180)
+    (pin "SDD[0..7]" input (at 322.58 91.44 180)
       (effects (font (size 1.27 1.27)) (justify left))
     )
