File: NeoGeoAES3_5.kicad_sch (KiCad schematic)
At the start: 0 parts

Commit message: Some tweaks
Other:
- company: (none) -> SNK
- title: (none) -> NeoGeo AES
Changed lines of the file:
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@@
 (kicad_sch (version 20230121) (generator eeschema)
   (paper "A3")
+  (title_block
+    (title "NeoGeo AES")
+    (date "2023-08-19")
+    (rev "3.5")
+    (company "SNK")
+    (comment 3 "https://github.com/Board-Folk")
+    (comment 4 "Recreated By The Board Folk Team")
+  )
   (junction (at 166.37 50.8) (diameter 0) (color 0 0 0 0)
   )

Commit message: Updates to PCB Move P2 Joystick Port Move Memory Card Move Holes at top right Silkscreen added Update Titles
Other:
- title: NeoGeo AES -> NeoGeo AES 3-5
Changed lines of the file:
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@@
   (paper "A3")
   (title_block
-    (title "NeoGeo AES")
-    (date "2023-08-19")
-    (rev "3.5")
+    (title "NeoGeo AES 3-5")
+    (date "2023-08-27")
+    (rev "BF1.1")
     (company "SNK")
     (comment 3 "https://github.com/Board-Folk")
