File: NeoGeoAES3_5.kicad_pcb (KiCad board)
At the start: 2 copper layers, 310 x 229.8 mm, 320 parts, among them CN1 CTRL1, CN2 CTRL2, CN3 DIN-8, CN4 AXC90020, CN5 AXC90020, CN6 Memory Card Interface, J1 BERR, J2 CUT DOG, J3 SMK S-G8043, J4 POWER JACK, Q101 2SC1815, Q102 2SC1815, Q11 C1815, Q12 A1015, Q13 A1442, SW1 RESET SWITCH, SW2 POWER SWITCH, T1 SH-302, U1 43256, U10 74LS273, U11 74LS05, U12 74LS06, U13 NEO-B1, U14 PST518B, U15 74LS244, U16 TC531000AP, U17 43256, U18 43256, U19 5863 / 5814, U2 43256, U20 5863 / 5814, U21 LSPC2, U22 NEO-D0, U23 6116, U24 Z80CPU, U26 YM3016D, U27 YM2610, U28 PC4741, U29 PC4741, U3 HD68HC000P, U32 CXA1145P, U33 74AS04, U34 NEO-E0, U35 74HC259, U36 27C1024, U37 LM2576T-5, U38 74HC32, U39 CX23065A, U4 NEO-C1, U5 NEO-G0, U6 4364, U7 4364, U8 74HC04, U80 74HC04, U9 74LS273, X1 24.167829MHz, X2 3.579545MHz

Commit message: Updated to Kicad 10
Parts:
- U19, U20: footprint 1_NeoGeoLibrary:DIP-28_W7.62mm-Dual -> 1_NeoGeoLibrary:DIP-28_W7.62mm
Connections:
- C45 pad 2: GND -> Net-(T1-AA)
- J4 pad 1: GND -> Net-(T1-AA)
- T1 pad 1: GND -> Net-(T1-AA)
- U21 pad 83: unconnected-(U21-NC-Pad83) -> GND
Routing:
- net Net-(T1-AA): track 0.00 -> 149.6 mm
- net GND: track 3341.4 -> 3205.7 mm
- added copper zone on B.Cu, net Net-(T1-AA)
- added copper zone on B.Cu, net unconnected-(RV1-Pad3)_1
Other:
- board text added: "The Board Folk Team 2026 Neogeo AES 3-5 Repo - BF1.5"
- board text removed: "The Board Folk Team 2024 Neogeo AES 3-5 Repo - BF1.4"
